File: Sandbox/Sandbox.kicad_sch (KiCad schematic)
At the start: 0 parts

Commit message: Test D-Latch Finished
Other:
- removed sheet NAND10
- removed sheet NAND11
Changed lines of the file:
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@@
-    )
-  )
-  (sheet (at 30.48 63.5) (size 24.13 12.7) (fields_autoplaced)
-    (stroke (width 0.1524) (type solid))
-    (fill (color 0 0 0 0.0000))
-    (property "Sheetname" "NAND10" (at 30.48 62.7884 0)
-      (effects (font (size 1.27 1.27)) (justify left bottom))
-    )
-    (property "Sheetfile" "nand.kicad_sch" (at 30.48 76.7846 0)
-      (effects (font (size 1.27 1.27)) (justify left top))
-    )
-    (pin "C" input (at 54.61 69.85 0)
-      (effects (font (size 1.27 1.27)) (justify right))
-    )
-    (pin "A" input (at 30.48 67.31 180)
-      (effects (font (size 1.27 1.27)) (justify left))
-    )
-    (pin "B" input (at 30.48 72.39 180)
-      (effects (font (size 1.27 1.27)) (justify left))
-    )
-    (instances
-      (project "Sandbox"
-        (path "/29877ccf-0b52-4099-b1b5-9309bc9469f9" (page "21"))
-      )
     )
   )
@@
       )
     )
-  )
-  (sheet (at 30.48 83.82) (size 24.13 12.7) (fields_autoplaced)
-    (stroke (width 0.1524) (type solid))
-    (fill (color 0 0 0 0.0000))
-    (property "Sheetname" "NAND11" (at 30.48 83.1084 0)
-      (effects (font (size 1.27 1.27)) (justify left bottom))
-    )
-    (property "Sheetfile" "nand.kicad_sch" (at 30.48 97.1046 0)
-      (effects (font (size 1.27 1.27)) (justify left top))
-    )
-    (pin "C" input (at 54.61 90.17 0)
-      (effects (font (size 1.27 1.27)) (justify right))
-    )
-    (pin "A" input (at 30.48 87.63 180)
-      (effects (font (size 1.27 1.27)) (justify left))
-    )
-    (pin "B" input (at 30.48 92.71 180)
-      (effects (font (size 1.27 1.27)) (justify left))
-    )
-    (instances
-      (project "Sandbox"
-        (path "/29877ccf-0b52-4099-b1b5-9309bc9469f9" (page "2"))
-      )
-    )
