File: Sandbox/D-Flip-Flop.kicad_sch (KiCad schematic)
At the start: 0 parts

Commit message: Test D-Latch Finished
Other:
- added sheet NAND15 (nand.kicad_sch)
- added sheet NAND16 (nand.kicad_sch)
Changed lines of the file:
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@@
     (instances
       (project "Sandbox"
-        (path "/29877ccf-0b52-4099-b1b5-9309bc9469f9/1964a911-d622-41af-9286-bec00cfc4577/e1952269-70f3-417e-afeb-be36723f1d92" (page "11"))
+        (path "/29877ccf-0b52-4099-b1b5-9309bc9469f9/1964a911-d622-41af-9286-bec00cfc4577/e1952269-70f3-417e-afeb-be36723f1d92" (page "4"))
+      )
+    )
+  )
+  (sheet (at 96.52 109.22) (size 24.13 12.7) (fields_autoplaced)
+    (stroke (width 0.1524) (type solid))
+    (fill (color 0 0 0 0.0000))
+    (property "Sheetname" "NAND16" (at 96.52 108.5084 0)
+      (effects (font (size 1.27 1.27)) (justify left bottom))
+    )
+    (property "Sheetfile" "nand.kicad_sch" (at 96.52 122.5046 0)
+      (effects (font (size 1.27 1.27)) (justify left top))
+    )
+    (pin "C" input (at 120.65 115.57 0)
+      (effects (font (size 1.27 1.27)) (justify right))
+    )
+    (pin "A" input (at 96.52 113.03 180)
+      (effects (font (size 1.27 1.27)) (justify left))
+    )
+    (pin "B" input (at 96.52 118.11 180)
+      (effects (font (size 1.27 1.27)) (justify left))
+    )
+    (instances
+      (project "Sandbox"
+        (path "/29877ccf-0b52-4099-b1b5-9309bc9469f9" (page "21"))
+        (path "/29877ccf-0b52-4099-b1b5-9309bc9469f9/1964a911-d622-41af-9286-bec00cfc4577/e1952269-70f3-417e-afeb-be36723f1d92/a1533095-cf41-4968-84d4-f6acc8b9549e/c3778304-4080-4c33-9045-4be924987a87" (page "2"))
+        (path "/29877ccf-0b52-4099-b1b5-9309bc9469f9/1964a911-d622-41af-9286-bec00cfc4577/e1952269-70f3-417e-afeb-be36723f1d92/06ab5ff7-08c5-4acf-a383-c54beac705bc/c3778304-4080-4c33-9045-4be924987a87" (page "9"))
+        (path "/29877ccf-0b52-4099-b1b5-9309bc9469f9/1964a911-d622-41af-9286-bec00cfc4577/e1952269-70f3-417e-afeb-be36723f1d92" (page "19"))
       )
     )
@@
       )
     )
+  )
+  (sheet (at 154.94 109.22) (size 24.13 12.7) (fields_autoplaced)
+    (stroke (width 0.1524) (type solid))
+    (fill (color 0 0 0 0.0000))
+    (property "Sheetname" "NAND15" (at 154.94 108.5084 0)
+      (effects (font (size 1.27 1.27)) (justify left bottom))
+    )
+    (property "Sheetfile" "nand.kicad_sch" (at 154.94 122.5046 0)
+      (effects (font (size 1.27 1.27)) (justify left top))
+    )
+    (pin "C" input (at 179.07 115.57 0)
+      (effects (font (size 1.27 1.27)) (justify right))
+    )
+    (pin "A" input (at 154.94 113.03 180)
+      (effects (font (size 1.27 1.27)) (justify left))
+    )
+    (pin "B" input (at 154.94 118.11 180)
+      (effects (font (size 1.27 1.27)) (justify left))
+    )
+    (instances
+      (project "Sandbox"
+        (path "/29877ccf-0b52-4099-b1b5-9309bc9469f9" (page "21"))
+        (path "/29877ccf-0b52-4099-b1b5-9309bc9469f9/1964a911-d622-41af-9286-bec00cfc4577/e1952269-70f3-417e-afeb-be36723f1d92/a1533095-cf41-4968-84d4-f6acc8b9549e/c3778304-4080-4c33-9045-4be924987a87" (page "2"))
+        (path "/29877ccf-0b52-4099-b1b5-9309bc9469f9/1964a911-d622-41af-9286-bec00cfc4577/e1952269-70f3-417e-afeb-be36723f1d92/06ab5ff7-08c5-4acf-a383-c54beac705bc/c3778304-4080-4c33-9045-4be924987a87" (page "9"))
+        (path "/29877ccf-0b52-4099-b1b5-9309bc9469f9/1964a911-d622-41af-9286-bec00cfc4577/e1952269-70f3-417e-afeb-be36723f1d92" (page "18"))
+      )
+    )

Commit message: Added Some stuff
Other:
- removed sheet D-Latch
- removed sheet NAND15
- removed sheet NAND16
Changed lines of the file:
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@@
-    )
-  )
-  (sheet (at 96.52 109.22) (size 24.13 12.7) (fields_autoplaced)
-    (stroke (width 0.1524) (type solid))
-    (fill (color 0 0 0 0.0000))
-    (property "Sheetname" "NAND16" (at 96.52 108.5084 0)
-      (effects (font (size 1.27 1.27)) (justify left bottom))
-    )
-    (property "Sheetfile" "nand.kicad_sch" (at 96.52 122.5046 0)
-      (effects (font (size 1.27 1.27)) (justify left top))
-    )
-    (pin "C" input (at 120.65 115.57 0)
-      (effects (font (size 1.27 1.27)) (justify right))
-    )
-    (pin "A" input (at 96.52 113.03 180)
-      (effects (font (size 1.27 1.27)) (justify left))
-    )
-    (pin "B" input (at 96.52 118.11 180)
-      (effects (font (size 1.27 1.27)) (justify left))
-    )
-    (instances
-      (project "Sandbox"
-        (path "/29877ccf-0b52-4099-b1b5-9309bc9469f9" (page "21"))
-        (path "/29877ccf-0b52-4099-b1b5-9309bc9469f9/1964a911-d622-41af-9286-bec00cfc4577/e1952269-70f3-417e-afeb-be36723f1d92/a1533095-cf41-4968-84d4-f6acc8b9549e/c3778304-4080-4c33-9045-4be924987a87" (page "2"))
-        (path "/29877ccf-0b52-4099-b1b5-9309bc9469f9/1964a911-d622-41af-9286-bec00cfc4577/e1952269-70f3-417e-afeb-be36723f1d92/06ab5ff7-08c5-4acf-a383-c54beac705bc/c3778304-4080-4c33-9045-4be924987a87" (page "9"))
-        (path "/29877ccf-0b52-4099-b1b5-9309bc9469f9/1964a911-d622-41af-9286-bec00cfc4577/e1952269-70f3-417e-afeb-be36723f1d92" (page "19"))
-      )
-    )
-  )
-  (sheet (at 128.27 77.47) (size 36.83 19.05) (fields_autoplaced)
-    (stroke (width 0.1524) (type solid))
-    (fill (color 0 0 0 0.0000))
-    (property "Sheetname" "D-Latch" (at 128.27 76.7584 0)
-      (effects (font (size 1.27 1.27)) (justify left bottom))
-    )
-    (property "Sheetfile" "D-Latch.kicad_sch" (at 128.27 97.1046 0)
-      (effects (font (size 1.27 1.27)) (justify left top))
-    )
-    (pin "Enable" input (at 128.27 92.71 180)
-      (effects (font (size 1.27 1.27)) (justify left))
-    )
-    (pin "Data" input (at 128.27 82.55 180)
-      (effects (font (size 1.27 1.27)) (justify left))
-    )
-    (pin "!Q" input (at 165.1 92.71 0)
-      (effects (font (size 1.27 1.27)) (justify right))
-    )
-    (pin "Q" input (at 165.1 82.55 0)
-      (effects (font (size 1.27 1.27)) (justify right))
-    )
-    (instances
-      (project "Sandbox"
-        (path "/29877ccf-0b52-4099-b1b5-9309bc9469f9/1964a911-d622-41af-9286-bec00cfc4577/e1952269-70f3-417e-afeb-be36723f1d92" (page "7"))
-      )
-    )
-  )
-  (sheet (at 154.94 109.22) (size 24.13 12.7) (fields_autoplaced)
-    (stroke (width 0.1524) (type solid))
-    (fill (color 0 0 0 0.0000))
-    (property "Sheetname" "NAND15" (at 154.94 108.5084 0)
-      (effects (font (size 1.27 1.27)) (justify left bottom))
-    )
-    (property "Sheetfile" "nand.kicad_sch" (at 154.94 122.5046 0)
-      (effects (font (size 1.27 1.27)) (justify left top))
-    )
-    (pin "C" input (at 179.07 115.57 0)
-      (effects (font (size 1.27 1.27)) (justify right))
-    )
-    (pin "A" input (at 154.94 113.03 180)
-      (effects (font (size 1.27 1.27)) (justify left))
-    )
-    (pin "B" input (at 154.94 118.11 180)
-      (effects (font (size 1.27 1.27)) (justify left))
-    )
-    (instances
-      (project "Sandbox"
-        (path "/29877ccf-0b52-4099-b1b5-9309bc9469f9" (page "21"))
-        (path "/29877ccf-0b52-4099-b1b5-9309bc9469f9/1964a911-d622-41af-9286-bec00cfc4577/e1952269-70f3-417e-afeb-be36723f1d92/a1533095-cf41-4968-84d4-f6acc8b9549e/c3778304-4080-4c33-9045-4be924987a87" (page "2"))
-        (path "/29877ccf-0b52-4099-b1b5-9309bc9469f9/1964a911-d622-41af-9286-bec00cfc4577/e1952269-70f3-417e-afeb-be36723f1d92/06ab5ff7-08c5-4acf-a383-c54beac705bc/c3778304-4080-4c33-9045-4be924987a87" (page "9"))
-        (path "/29877ccf-0b52-4099-b1b5-9309bc9469f9/1964a911-d622-41af-9286-bec00cfc4577/e1952269-70f3-417e-afeb-be36723f1d92" (page "18"))
-      )
     )
   )
