File: Sandbox/D-Latch.kicad_sch (KiCad schematic)
At the start: 0 parts

Commit message: Test D-Latch Finished
Other:
- added sheet NAND12 (nand.kicad_sch)
- added sheet NAND13 (nand.kicad_sch)
- added sheet NAND14 (nand.kicad_sch)
Changed lines of the file:
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@@
     (effects (font (size 1.27 1.27)) (justify left))
+  )
+  (sheet (at 133.35 85.09) (size 24.13 12.7) (fields_autoplaced)
+    (stroke (width 0.1524) (type solid))
+    (fill (color 0 0 0 0.0000))
+    (property "Sheetname" "NAND13" (at 133.35 84.3784 0)
+      (effects (font (size 1.27 1.27)) (justify left bottom))
+    )
+    (property "Sheetfile" "nand.kicad_sch" (at 133.35 98.3746 0)
+      (effects (font (size 1.27 1.27)) (justify left top))
+    )
+    (pin "C" input (at 157.48 91.44 0)
+      (effects (font (size 1.27 1.27)) (justify right))
+    )
+    (pin "A" input (at 133.35 88.9 180)
+      (effects (font (size 1.27 1.27)) (justify left))
+    )
+    (pin "B" input (at 133.35 93.98 180)
+      (effects (font (size 1.27 1.27)) (justify left))
+    )
+    (instances
+      (project "Sandbox"
+        (path "/29877ccf-0b52-4099-b1b5-9309bc9469f9" (page "21"))
+        (path "/29877ccf-0b52-4099-b1b5-9309bc9469f9/1964a911-d622-41af-9286-bec00cfc4577/e1952269-70f3-417e-afeb-be36723f1d92/a1533095-cf41-4968-84d4-f6acc8b9549e/c3778304-4080-4c33-9045-4be924987a87" (page "2"))
+        (path "/29877ccf-0b52-4099-b1b5-9309bc9469f9/1964a911-d622-41af-9286-bec00cfc4577/e1952269-70f3-417e-afeb-be36723f1d92/06ab5ff7-08c5-4acf-a383-c54beac705bc/c3778304-4080-4c33-9045-4be924987a87" (page "9"))
+        (path "/29877ccf-0b52-4099-b1b5-9309bc9469f9/1964a911-d622-41af-9286-bec00cfc4577/e1952269-70f3-417e-afeb-be36723f1d92/06ab5ff7-08c5-4acf-a383-c54beac705bc" (page "14"))
+        (path "/29877ccf-0b52-4099-b1b5-9309bc9469f9/1964a911-d622-41af-9286-bec00cfc4577/e1952269-70f3-417e-afeb-be36723f1d92/a1533095-cf41-4968-84d4-f6acc8b9549e" (page "15"))
+      )
+    )
+  )
+  (sheet (at 85.09 87.63) (size 24.13 12.7) (fields_autoplaced)
+    (stroke (width 0.1524) (type solid))
+    (fill (color 0 0 0 0.0000))
+    (property "Sheetname" "NAND14" (at 85.09 86.9184 0)
+      (effects (font (size 1.27 1.27)) (justify left bottom))
+    )
+    (property "Sheetfile" "nand.kicad_sch" (at 85.09 100.9146 0)
+      (effects (font (size 1.27 1.27)) (justify left top))
+    )
+    (pin "C" input (at 109.22 93.98 0)
+      (effects (font (size 1.27 1.27)) (justify right))
+    )
+    (pin "A" input (at 85.09 91.44 180)
+      (effects (font (size 1.27 1.27)) (justify left))
+    )
+    (pin "B" input (at 85.09 96.52 180)
+      (effects (font (size 1.27 1.27)) (justify left))
+    )
+    (instances
+      (project "Sandbox"
+        (path "/29877ccf-0b52-4099-b1b5-9309bc9469f9" (page "21"))
+        (path "/29877ccf-0b52-4099-b1b5-9309bc9469f9/1964a911-d622-41af-9286-bec00cfc4577/e1952269-70f3-417e-afeb-be36723f1d92/a1533095-cf41-4968-84d4-f6acc8b9549e/c3778304-4080-4c33-9045-4be924987a87" (page "2"))
+        (path "/29877ccf-0b52-4099-b1b5-9309bc9469f9/1964a911-d622-41af-9286-bec00cfc4577/e1952269-70f3-417e-afeb-be36723f1d92/06ab5ff7-08c5-4acf-a383-c54beac705bc/c3778304-4080-4c33-9045-4be924987a87" (page "9"))
+        (path "/29877ccf-0b52-4099-b1b5-9309bc9469f9/1964a911-d622-41af-9286-bec00cfc4577/e1952269-70f3-417e-afeb-be36723f1d92/06ab5ff7-08c5-4acf-a383-c54beac705bc" (page "16"))
+        (path "/29877ccf-0b52-4099-b1b5-9309bc9469f9/1964a911-d622-41af-9286-bec00cfc4577/e1952269-70f3-417e-afeb-be36723f1d92/a1533095-cf41-4968-84d4-f6acc8b9549e" (page "17"))
+      )
+    )
   )
   (sheet (at 173.99 63.5) (size 34.29 13.97) (fields_autoplaced)
@@
       (project "Sandbox"
         (path "/29877ccf-0b52-4099-b1b5-9309bc9469f9/1964a911-d622-41af-9286-bec00cfc4577/e1952269-70f3-417e-afeb-be36723f1d92/a1533095-cf41-4968-84d4-f6acc8b9549e" (page "8"))
-        (path "/29877ccf-0b52-4099-b1b5-9309bc9469f9/1964a911-d622-41af-9286-bec00cfc4577/e1952269-70f3-417e-afeb-be36723f1d92/6ec43859-8a9a-4225-81ff-d535bdc822af" (page "15"))
+        (path "/29877ccf-0b52-4099-b1b5-9309bc9469f9/1964a911-d622-41af-9286-bec00cfc4577/e1952269-70f3-417e-afeb-be36723f1d92/06ab5ff7-08c5-4acf-a383-c54beac705bc" (page "11"))
       )
     )
+  )
+  (sheet (at 132.08 53.34) (size 24.13 12.7) (fields_autoplaced)
+    (stroke (width 0.1524) (type solid))
+    (fill (color 0 0 0 0.0000))
+    (property "Sheetname" "NAND12" (at 132.08 52.6284 0)
+      (effects (font (size 1.27 1.27)) (justify left bottom))
+    )
+    (property "Sheetfile" "nand.kicad_sch" (at 132.08 66.6246 0)
+      (effects (font (size 1.27 1.27)) (justify left top))
+    )
+    (pin "C" input (at 156.21 59.69 0)
+      (effects (font (size 1.27 1.27)) (justify right))
+    )
+    (pin "A" input (at 132.08 57.15 180)
+      (effects (font (size 1.27 1.27)) (justify left))
+    )
+    (pin "B" input (at 132.08 62.23 180)
+      (effects (font (size 1.27 1.27)) (justify left))
+    )
+    (instances
+      (project "Sandbox"
+        (path "/29877ccf-0b52-4099-b1b5-9309bc9469f9" (page "21"))
+        (path "/29877ccf-0b52-4099-b1b5-9309bc9469f9/1964a911-d622-41af-9286-bec00cfc4577/e1952269-70f3-417e-afeb-be36723f1d92/a1533095-cf41-4968-84d4-f6acc8b9549e/c3778304-4080-4c33-9045-4be924987a87" (page "2"))
+        (path "/29877ccf-0b52-4099-b1b5-9309bc9469f9/1964a911-d622-41af-9286-bec00cfc4577/e1952269-70f3-417e-afeb-be36723f1d92/06ab5ff7-08c5-4acf-a383-c54beac705bc/c3778304-4080-4c33-9045-4be924987a87" (page "9"))
+        (path "/29877ccf-0b52-4099-b1b5-9309bc9469f9/1964a911-d622-41af-9286-bec00cfc4577/e1952269-70f3-417e-afeb-be36723f1d92/06ab5ff7-08c5-4acf-a383-c54beac705bc" (page "12"))
+        (path "/29877ccf-0b52-4099-b1b5-9309bc9469f9/1964a911-d622-41af-9286-bec00cfc4577/e1952269-70f3-417e-afeb-be36723f1d92/a1533095-cf41-4968-84d4-f6acc8b9549e" (page "13"))
+      )
+    )

Commit message: Added Some stuff
Other:
- removed sheet NAND12
- removed sheet NAND13
- removed sheet NAND14
Changed lines of the file:
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@@
     (effects (font (size 1.27 1.27)) (justify left))
-  )
-  (sheet (at 133.35 85.09) (size 24.13 12.7) (fields_autoplaced)
-    (stroke (width 0.1524) (type solid))
-    (fill (color 0 0 0 0.0000))
-    (property "Sheetname" "NAND13" (at 133.35 84.3784 0)
-      (effects (font (size 1.27 1.27)) (justify left bottom))
-    )
-    (property "Sheetfile" "nand.kicad_sch" (at 133.35 98.3746 0)
-      (effects (font (size 1.27 1.27)) (justify left top))
-    )
-    (pin "C" input (at 157.48 91.44 0)
-      (effects (font (size 1.27 1.27)) (justify right))
-    )
-    (pin "A" input (at 133.35 88.9 180)
-      (effects (font (size 1.27 1.27)) (justify left))
-    )
-    (pin "B" input (at 133.35 93.98 180)
-      (effects (font (size 1.27 1.27)) (justify left))
-    )
-    (instances
-      (project "Sandbox"
-        (path "/29877ccf-0b52-4099-b1b5-9309bc9469f9" (page "21"))
-        (path "/29877ccf-0b52-4099-b1b5-9309bc9469f9/1964a911-d622-41af-9286-bec00cfc4577/e1952269-70f3-417e-afeb-be36723f1d92/a1533095-cf41-4968-84d4-f6acc8b9549e/c3778304-4080-4c33-9045-4be924987a87" (page "2"))
-        (path "/29877ccf-0b52-4099-b1b5-9309bc9469f9/1964a911-d622-41af-9286-bec00cfc4577/e1952269-70f3-417e-afeb-be36723f1d92/06ab5ff7-08c5-4acf-a383-c54beac705bc/c3778304-4080-4c33-9045-4be924987a87" (page "9"))
-        (path "/29877ccf-0b52-4099-b1b5-9309bc9469f9/1964a911-d622-41af-9286-bec00cfc4577/e1952269-70f3-417e-afeb-be36723f1d92/06ab5ff7-08c5-4acf-a383-c54beac705bc" (page "14"))
-        (path "/29877ccf-0b52-4099-b1b5-9309bc9469f9/1964a911-d622-41af-9286-bec00cfc4577/e1952269-70f3-417e-afeb-be36723f1d92/a1533095-cf41-4968-84d4-f6acc8b9549e" (page "15"))
-      )
-    )
-  )
-  (sheet (at 85.09 87.63) (size 24.13 12.7) (fields_autoplaced)
-    (stroke (width 0.1524) (type solid))
-    (fill (color 0 0 0 0.0000))
-    (property "Sheetname" "NAND14" (at 85.09 86.9184 0)
-      (effects (font (size 1.27 1.27)) (justify left bottom))
-    )
-    (property "Sheetfile" "nand.kicad_sch" (at 85.09 100.9146 0)
-      (effects (font (size 1.27 1.27)) (justify left top))
-    )
-    (pin "C" input (at 109.22 93.98 0)
-      (effects (font (size 1.27 1.27)) (justify right))
-    )
-    (pin "A" input (at 85.09 91.44 180)
-      (effects (font (size 1.27 1.27)) (justify left))
-    )
-    (pin "B" input (at 85.09 96.52 180)
-      (effects (font (size 1.27 1.27)) (justify left))
-    )
-    (instances
-      (project "Sandbox"
-        (path "/29877ccf-0b52-4099-b1b5-9309bc9469f9" (page "21"))
-        (path "/29877ccf-0b52-4099-b1b5-9309bc9469f9/1964a911-d622-41af-9286-bec00cfc4577/e1952269-70f3-417e-afeb-be36723f1d92/a1533095-cf41-4968-84d4-f6acc8b9549e/c3778304-4080-4c33-9045-4be924987a87" (page "2"))
-        (path "/29877ccf-0b52-4099-b1b5-9309bc9469f9/1964a911-d622-41af-9286-bec00cfc4577/e1952269-70f3-417e-afeb-be36723f1d92/06ab5ff7-08c5-4acf-a383-c54beac705bc/c3778304-4080-4c33-9045-4be924987a87" (page "9"))
-        (path "/29877ccf-0b52-4099-b1b5-9309bc9469f9/1964a911-d622-41af-9286-bec00cfc4577/e1952269-70f3-417e-afeb-be36723f1d92/06ab5ff7-08c5-4acf-a383-c54beac705bc" (page "16"))
-        (path "/29877ccf-0b52-4099-b1b5-9309bc9469f9/1964a911-d622-41af-9286-bec00cfc4577/e1952269-70f3-417e-afeb-be36723f1d92/a1533095-cf41-4968-84d4-f6acc8b9549e" (page "17"))
-      )
-    )
   )
   (sheet (at 173.99 63.5) (size 34.29 13.97) (fields_autoplaced)
@@
     (instances
       (project "Sandbox"
-        (path "/29877ccf-0b52-4099-b1b5-9309bc9469f9/1964a911-d622-41af-9286-bec00cfc4577/e1952269-70f3-417e-afeb-be36723f1d92/a1533095-cf41-4968-84d4-f6acc8b9549e" (page "8"))
         (path "/29877ccf-0b52-4099-b1b5-9309bc9469f9/1964a911-d622-41af-9286-bec00cfc4577/e1952269-70f3-417e-afeb-be36723f1d92/06ab5ff7-08c5-4acf-a383-c54beac705bc" (page "11"))
       )
     )
-  )
-  (sheet (at 132.08 53.34) (size 24.13 12.7) (fields_autoplaced)
-    (stroke (width 0.1524) (type solid))
-    (fill (color 0 0 0 0.0000))
-    (property "Sheetname" "NAND12" (at 132.08 52.6284 0)
-      (effects (font (size 1.27 1.27)) (justify left bottom))
-    )
-    (property "Sheetfile" "nand.kicad_sch" (at 132.08 66.6246 0)
-      (effects (font (size 1.27 1.27)) (justify left top))
-    )
-    (pin "C" input (at 156.21 59.69 0)
-      (effects (font (size 1.27 1.27)) (justify right))
-    )
-    (pin "A" input (at 132.08 57.15 180)
-      (effects (font (size 1.27 1.27)) (justify left))
-    )
-    (pin "B" input (at 132.08 62.23 180)
-      (effects (font (size 1.27 1.27)) (justify left))
-    )
-    (instances
-      (project "Sandbox"
-        (path "/29877ccf-0b52-4099-b1b5-9309bc9469f9" (page "21"))
-        (path "/29877ccf-0b52-4099-b1b5-9309bc9469f9/1964a911-d622-41af-9286-bec00cfc4577/e1952269-70f3-417e-afeb-be36723f1d92/a1533095-cf41-4968-84d4-f6acc8b9549e/c3778304-4080-4c33-9045-4be924987a87" (page "2"))
-        (path "/29877ccf-0b52-4099-b1b5-9309bc9469f9/1964a911-d622-41af-9286-bec00cfc4577/e1952269-70f3-417e-afeb-be36723f1d92/06ab5ff7-08c5-4acf-a383-c54beac705bc/c3778304-4080-4c33-9045-4be924987a87" (page "9"))
-        (path "/29877ccf-0b52-4099-b1b5-9309bc9469f9/1964a911-d622-41af-9286-bec00cfc4577/e1952269-70f3-417e-afeb-be36723f1d92/06ab5ff7-08c5-4acf-a383-c54beac705bc" (page "12"))
-        (path "/29877ccf-0b52-4099-b1b5-9309bc9469f9/1964a911-d622-41af-9286-bec00cfc4577/e1952269-70f3-417e-afeb-be36723f1d92/a1533095-cf41-4968-84d4-f6acc8b9549e" (page "13"))
-      )
-    )
