File: Sandbox/Register.kicad_sch (KiCad schematic)
At the start: 6 parts, among them SW1 SW_Push_Dual, SW2 SW_Push_Dual

Commit message: Test D-Latch Finished
Connections:
- net +5V renamed VCC
Changed lines of the file:
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@@
 (kicad_sch (version 20230121) (generator eeschema)
   (paper "A4")
+  (junction (at 156.21 68.58) (diameter 0) (color 0 0 0 0)
+  )
+  (junction (at 63.5 68.58) (diameter 0) (color 0 0 0 0)
+  )
+  (junction (at 73.66 69.85) (diameter 0) (color 0 0 0 0)
+  )
+  (junction (at 69.85 85.09) (diameter 0) (color 0 0 0 0)
+  )
   (junction (at 59.69 85.09) (diameter 0) (color 0 0 0 0)
-  )
-  (junction (at 156.21 68.58) (diameter 0) (color 0 0 0 0)
-  )
-  (junction (at 73.66 69.85) (diameter 0) (color 0 0 0 0)
-  )
-  (junction (at 63.5 68.58) (diameter 0) (color 0 0 0 0)
-  )
-  (junction (at 69.85 85.09) (diameter 0) (color 0 0 0 0)
   )
   (wire (pts (xy 148.59 68.58) (xy 143.51 68.58))
@@
     )
   )
-  (symbol (lib_id "power:+5V") (at 59.69 85.09 90) (unit 1)
-    (in_bom yes) (on_board yes) (dnp no) (fields_autoplaced)
-    (property "Reference" "#PWR027" (at 63.5 85.09 0)
-      (effects (font (size 1.27 1.27)) hide)
-    )
-    (property "Value" "+5V" (at 55.88 85.09 90)
-      (effects (font (size 1.27 1.27)) (justify left))
-    )
-    (property "Footprint" "" (at 59.69 85.09 0)
-      (effects (font (size 1.27 1.27)) hide)
-    )
-    (property "Datasheet" "" (at 59.69 85.09 0)
-      (effects (font (size 1.27 1.27)) hide)
-    )
-    (pin "1")
-    (instances
-      (project "Sandbox"
-        (path "/29877ccf-0b52-4099-b1b5-9309bc9469f9/1964a911-d622-41af-9286-bec00cfc4577"
-          (reference "#PWR027") (unit 1)
-        )
-      )
-    )
-  )
   (symbol (lib_id "Device:LED") (at 139.7 78.74 180) (unit 1)
     (in_bom yes) (on_board yes) (dnp no) (fields_autoplaced)
@@
     )
   )
-  (symbol (lib_id "power:+5V") (at 63.5 68.58 90) (unit 1)
+  (symbol (lib_id "power:VCC") (at 63.5 68.58 90) (unit 1)
     (in_bom yes) (on_board yes) (dnp no) (fields_autoplaced)
     (property "Reference" "#PWR026" (at 67.31 68.58 0)
       (effects (font (size 1.27 1.27)) hide)
     )
-    (property "Value" "+5V" (at 59.69 68.58 90)
+    (property "Value" "VCC" (at 59.69 68.58 90)
       (effects (font (size 1.27 1.27)) (justify left))
     )
@@
         )
       )
+    )
+  )
+  (symbol (lib_id "power:VCC") (at 59.69 85.09 90) (unit 1)
+    (in_bom yes) (on_board yes) (dnp no) (fields_autoplaced)
+    (property "Reference" "#PWR027" (at 63.5 85.09 0)
+      (effects (font (size 1.27 1.27)) hide)
+    )
+    (property "Value" "VCC" (at 55.88 85.09 90)
+      (effects (font (size 1.27 1.27)) (justify left))
+    )
+    (property "Footprint" "" (at 59.69 85.09 0)
+      (effects (font (size 1.27 1.27)) hide)
+    )
+    (property "Datasheet" "" (at 59.69 85.09 0)
+      (effects (font (size 1.27 1.27)) hide)
+    )
+    (pin "1")
+    (instances
+      (project "Sandbox"
+        (path "/29877ccf-0b52-4099-b1b5-9309bc9469f9/1964a911-d622-41af-9286-bec00cfc4577"
+          (reference "#PWR027") (unit 1)
+        )
+      )

Commit message: Added Some stuff
Parts:
- removed D1, D2: LED, LED_THT:LED_D5.0mm_Clear, symbol Device:LED
- removed R37, R38: 1000, Resistor_THT:R_Axial_DIN0207_L6.3mm_D2.5mm_P10.16mm_Horizontal, symbol Device:R
- removed SW1, SW2: SW_Push_Dual, Button_Switch_THT:SW_PUSH_6mm, symbol Switch:SW_Push_Dual
Changed lines of the file:
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@@
 (kicad_sch (version 20230121) (generator eeschema)
   (paper "A4")
-  (junction (at 156.21 68.58) (diameter 0) (color 0 0 0 0)
-  )
-  (junction (at 63.5 68.58) (diameter 0) (color 0 0 0 0)
-  )
   (junction (at 73.66 69.85) (diameter 0) (color 0 0 0 0)
-  )
-  (junction (at 69.85 85.09) (diameter 0) (color 0 0 0 0)
-  )
-  (junction (at 59.69 85.09) (diameter 0) (color 0 0 0 0)
   )
   (wire (pts (xy 148.59 68.58) (xy 143.51 68.58))
@@
     (stroke (width 0) (type default))
   )
-  (wire (pts (xy 69.85 85.09) (xy 69.85 90.17))
+  (wire (pts (xy 69.85 81.28) (xy 69.85 90.17))
     (stroke (width 0) (type default))
   )
@@
     (stroke (width 0) (type default))
   )
-  (wire (pts (xy 148.59 78.74) (xy 143.51 78.74))
-    (stroke (width 0) (type default))
-  )
-  (wire (pts (xy 69.85 81.28) (xy 69.85 85.09))
-    (stroke (width 0) (type default))
-  )
-  (symbol (lib_id "Device:LED") (at 139.7 68.58 180) (unit 1)
-    (in_bom yes) (on_board yes) (dnp no) (fields_autoplaced)
-    (property "Reference" "D1" (at 141.2875 60.96 0)
-      (effects (font (size 1.27 1.27)))
-    )
-    (property "Value" "LED" (at 141.2875 63.5 0)
-      (effects (font (size 1.27 1.27)))
-    )
-    (property "Footprint" "LED_THT:LED_D5.0mm_Clear" (at 139.7 68.58 0)
-      (effects (font (size 1.27 1.27)) hide)
-    )
-    (property "Datasheet" "~" (at 139.7 68.58 0)
-      (effects (font (size 1.27 1.27)) hide)
-    )
-    (pin "1")
-    (pin "2")
-    (instances
-      (project "Sandbox"
-        (path "/29877ccf-0b52-4099-b1b5-9309bc9469f9/1964a911-d622-41af-9286-bec00cfc4577"
-          (reference "D1") (unit 1)
-        )
-      )
-    )
-  )
-  (symbol (lib_id "Switch:SW_Push_Dual") (at 68.58 68.58 0) (unit 1)
-    (in_bom yes) (on_board yes) (dnp no) (fields_autoplaced)
-    (property "Reference" "SW1" (at 68.58 60.96 0)
-      (effects (font (size 1.27 1.27)))
-    )
-    (property "Value" "SW_Push_Dual" (at 68.58 63.5 0)
-      (effects (font (size 1.27 1.27)))
-    )
-    (property "Footprint" "Button_Switch_THT:SW_PUSH_6mm" (at 68.58 63.5 0)
-      (effects (font (size 1.27 1.27)) hide)
-    )
-    (property "Datasheet" "~" (at 68.58 63.5 0)
-      (effects (font (size 1.27 1.27)) hide)
-    )
-    (pin "1")
-    (pin "2")
-    (pin "3")
-    (pin "4")
-    (instances
-      (project "Sandbox"
-        (path "/29877ccf-0b52-4099-b1b5-9309bc9469f9/1964a911-d622-41af-9286-bec00cfc4577"
-          (reference "SW1") (unit 1)
-        )
-      )
-    )
-  )
   (symbol (lib_id "power:GND") (at 168.91 68.58 90) (unit 1)
     (in_bom yes) (on_board yes) (dnp no) (fields_autoplaced)
@@
         (path "/29877ccf-0b52-4099-b1b5-9309bc9469f9/1964a911-d622-41af-9286-bec00cfc4577"
           (reference "#PWR025") (unit 1)
-        )
-      )
-    )
-  )
-  (symbol (lib_id "Device:LED") (at 139.7 78.74 180) (unit 1)
-    (in_bom yes) (on_board yes) (dnp no) (fields_autoplaced)
-    (property "Reference" "D2" (at 141.2875 71.12 0)
-      (effects (font (size 1.27 1.27)))
-    )
-    (property "Value" "LED" (at 141.2875 73.66 0)
-      (effects (font (size 1.27 1.27)))
-    )
-    (property "Footprint" "LED_THT:LED_D5.0mm_Clear" (at 139.7 78.74 0)
-      (effects (font (size 1.27 1.27)) hide)
-    )
-    (property "Datasheet" "~" (at 139.7 78.74 0)
-      (effects (font (size 1.27 1.27)) hide)
-    )
-    (pin "1")
-    (pin "2")
-    (instances
-      (project "Sandbox"
-        (path "/29877ccf-0b52-4099-b1b5-9309bc9469f9/1964a911-d622-41af-9286-bec00cfc4577"
-          (reference "D2") (unit 1)
         )
       )
@@
     )
   )
-  (symbol (lib_id "Switch:SW_Push_Dual") (at 64.77 85.09 0) (unit 1)
-    (in_bom yes) (on_board yes) (dnp no) (fields_autoplaced)
-    (property "Reference" "SW2" (at 64.77 77.47 0)
-      (effects (font (size 1.27 1.27)))
-    )
-    (property "Value" "SW_Push_Dual" (at 64.77 80.01 0)
-      (effects (font (size 1.27 1.27)))
-    )
-    (property "Footprint" "Button_Switch_THT:SW_PUSH_6mm" (at 64.77 80.01 0)
-      (effects (font (size 1.27 1.27)) hide)
-    )
-    (property "Datasheet" "~" (at 64.77 80.01 0)
-      (effects (font (size 1.27 1.27)) hide)
-    )
-    (pin "1")
-    (pin "2")
-    (pin "3")
-    (pin "4")
-    (instances
-      (project "Sandbox"
-        (path "/29877ccf-0b52-4099-b1b5-9309bc9469f9/1964a911-d622-41af-9286-bec00cfc4577"
-          (reference "SW2") (unit 1)
-        )
-      )
-    )
-  )
   (symbol (lib_id "power:VCC") (at 59.69 85.09 90) (unit 1)
     (in_bom yes) (on_board yes) (dnp no) (fields_autoplaced)
@@
         )
       )
-    )
-  )
-  (symbol (lib_id "Device:R") (at 152.4 68.58 90) (unit 1)
-    (in_bom yes) (on_board yes) (dnp no) (fields_autoplaced)
-    (property "Reference" "R37" (at 152.4 62.23 90)
-      (effects (font (size 1.27 1.27)))
-    )
-    (property "Value" "1000" (at 152.4 64.77 90)
-      (effects (font (size 1.27 1.27)))
-    )
-    (property "Footprint" "Resistor_THT:R_Axial_DIN0207_L6.3mm_D2.5mm_P10.16mm_Horizontal" (at 152.4 70.358 90)
-      (effects (font (size 1.27 1.27)) hide)
-    )
-    (property "Datasheet" "~" (at 152.4 68.58 0)
-      (effects (font (size 1.27 1.27)) hide)
-    )
-    (pin "1")
-    (pin "2")
-    (instances
-      (project "Sandbox"
-        (path "/29877ccf-0b52-4099-b1b5-9309bc9469f9/1964a911-d622-41af-9286-bec00cfc4577"
-          (reference "R37") (unit 1)
-        )
-      )
-    )
-  )
-  (symbol (lib_id "Device:R") (at 152.4 78.74 90) (unit 1)
-    (in_bom yes) (on_board yes) (dnp no) (fields_autoplaced)
-    (property "Reference" "R38" (at 152.4 72.39 90)
-      (effects (font (size 1.27 1.27)))
-    )
-    (property "Value" "1000" (at 152.4 74.93 90)
-      (effects (font (size 1.27 1.27)))
-    )
-    (property "Footprint" "Resistor_THT:R_Axial_DIN0207_L6.3mm_D2.5mm_P10.16mm_Horizontal" (at 152.4 80.518 90)
-      (effects (font (size 1.27 1.27)) hide)
-    )
-    (property "Datasheet" "~" (at 152.4 78.74 0)
-      (effects (font (size 1.27 1.27)) hide)
-    )
-    (pin "1")
-    (pin "2")
-    (instances
-      (project "Sandbox"
-        (path "/29877ccf-0b52-4099-b1b5-9309bc9469f9/1964a911-d622-41af-9286-bec00cfc4577"
-          (reference "R38") (unit 1)
-        )
-      )
