File: Sandbox/SR-Latch.kicad_sch (KiCad schematic)
At the start: 0 parts

Commit message: Test D-Latch Finished
Other:
- added sheet NAND10 (nand.kicad_sch)
- added sheet NAND11 (nand.kicad_sch)
Changed lines of the file:
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@@
     (effects (font (size 1.27 1.27)) (justify left))
   )
+  (sheet (at 81.28 73.66) (size 24.13 12.7) (fields_autoplaced)
+    (stroke (width 0.1524) (type solid))
+    (fill (color 0 0 0 0.0000))
+    (property "Sheetname" "NAND11" (at 81.28 72.9484 0)
+      (effects (font (size 1.27 1.27)) (justify left bottom))
+    )
+    (property "Sheetfile" "nand.kicad_sch" (at 81.28 86.9446 0)
+      (effects (font (size 1.27 1.27)) (justify left top))
+    )
+    (pin "C" input (at 105.41 80.01 0)
+      (effects (font (size 1.27 1.27)) (justify right))
+    )
+    (pin "A" input (at 81.28 77.47 180)
+      (effects (font (size 1.27 1.27)) (justify left))
+    )
+    (pin "B" input (at 81.28 82.55 180)
+      (effects (font (size 1.27 1.27)) (justify left))
+    )
+    (instances
+      (project "Sandbox"
+        (path "/29877ccf-0b52-4099-b1b5-9309bc9469f9" (page "21"))
+        (path "/29877ccf-0b52-4099-b1b5-9309bc9469f9/1964a911-d622-41af-9286-bec00cfc4577/e1952269-70f3-417e-afeb-be36723f1d92/a1533095-cf41-4968-84d4-f6acc8b9549e/c3778304-4080-4c33-9045-4be924987a87" (page "3"))
+        (path "/29877ccf-0b52-4099-b1b5-9309bc9469f9/1964a911-d622-41af-9286-bec00cfc4577/e1952269-70f3-417e-afeb-be36723f1d92/06ab5ff7-08c5-4acf-a383-c54beac705bc/c3778304-4080-4c33-9045-4be924987a87" (page "10"))
+      )
+    )
+  )
+  (sheet (at 81.28 46.99) (size 24.13 12.7) (fields_autoplaced)
+    (stroke (width 0.1524) (type solid))
+    (fill (color 0 0 0 0.0000))
+    (property "Sheetname" "NAND10" (at 81.28 46.2784 0)
+      (effects (font (size 1.27 1.27)) (justify left bottom))
+    )
+    (property "Sheetfile" "nand.kicad_sch" (at 81.28 60.2746 0)
+      (effects (font (size 1.27 1.27)) (justify left top))
+    )
+    (pin "C" input (at 105.41 53.34 0)
+      (effects (font (size 1.27 1.27)) (justify right))
+    )
+    (pin "A" input (at 81.28 50.8 180)
+      (effects (font (size 1.27 1.27)) (justify left))
+    )
+    (pin "B" input (at 81.28 55.88 180)
+      (effects (font (size 1.27 1.27)) (justify left))
+    )
+    (instances
+      (project "Sandbox"
+        (path "/29877ccf-0b52-4099-b1b5-9309bc9469f9" (page "21"))
+        (path "/29877ccf-0b52-4099-b1b5-9309bc9469f9/1964a911-d622-41af-9286-bec00cfc4577/e1952269-70f3-417e-afeb-be36723f1d92/a1533095-cf41-4968-84d4-f6acc8b9549e/c3778304-4080-4c33-9045-4be924987a87" (page "2"))
+        (path "/29877ccf-0b52-4099-b1b5-9309bc9469f9/1964a911-d622-41af-9286-bec00cfc4577/e1952269-70f3-417e-afeb-be36723f1d92/06ab5ff7-08c5-4acf-a383-c54beac705bc/c3778304-4080-4c33-9045-4be924987a87" (page "9"))
+      )
+    )
+  )
 )

Commit message: Added Some stuff
Parts:
- added D2: LED, LED_THT:LED_D5.0mm_Clear, symbol Device:LED
- added R38: 1000, Resistor_THT:R_Axial_DIN0207_L6.3mm_D2.5mm_P10.16mm_Horizontal, symbol Device:R
- added SW2 (x2): SW_Push_Dual, Button_Switch_THT:SW_PUSH_6mm, symbol Switch:SW_Push_Dual
Connections:
- new net: D2.1 (K), R38.1
- new net GND: R38.2
- new net NAND11/A: SW2.2, SW2.4
- new net NAND11/B: SW2.2
- new net NAND11/C: D2.2 (A)
- new net VCC: SW2.1, SW2.1, SW2.3
Other:
- removed sheet NAND10
