File: Sandbox/Sandbox.kicad_pcb (KiCad board)
At the start: 2 copper layers, 18 parts, among them Q1 2N3904, Q2 2N3904, Q3 2N3904, Q37 2N3904, Q38 2N3904, Q39 2N3904, SW1 SW_Push_Dual, SW2 SW_Push_Dual

Commit message: Test D-Latch Finished
Parts:
- removed Q37, Q38, Q39: 2N3904, Package_TO_SOT_THT:TO-92_Inline
- removed R39, R40: 1000, Resistor_THT:R_Axial_DIN0207_L6.3mm_D2.5mm_P10.16mm_Horizontal
- removed R41: 100, Resistor_THT:R_Axial_DIN0207_L6.3mm_D2.5mm_P10.16mm_Horizontal
- added Q10: 2N3904, Package_TO_SOT_THT:TO-92_Inline, F.Cu at (700.3, 449.8)
- added Q11: 2N3904, Package_TO_SOT_THT:TO-92_Inline, F.Cu at (700.3, 455.3)
- added Q12: 2N3904, Package_TO_SOT_THT:TO-92_Inline, F.Cu at (707.2, 449.8)
- added Q13: 2N3904, Package_TO_SOT_THT:TO-92_Inline, F.Cu at (631.8, 414.0)
- added Q14: 2N3904, Package_TO_SOT_THT:TO-92_Inline, F.Cu at (631.8, 419.5)
- added Q15: 2N3904, Package_TO_SOT_THT:TO-92_Inline, F.Cu at (638.6, 414.0)
- added Q16: 2N3904, Package_TO_SOT_THT:TO-92_Inline, F.Cu at (440.6, 413.6)
- added Q17: 2N3904, Package_TO_SOT_THT:TO-92_Inline, F.Cu at (440.6, 419.1)
- added Q18: 2N3904, Package_TO_SOT_THT:TO-92_Inline, F.Cu at (447.4, 413.6)
- added Q19: 2N3904, Package_TO_SOT_THT:TO-92_Inline, F.Cu at (629.2, 450.7)
- added Q20: 2N3904, Package_TO_SOT_THT:TO-92_Inline, F.Cu at (629.2, 456.2)
- added Q21: 2N3904, Package_TO_SOT_THT:TO-92_Inline, F.Cu at (636.1, 450.7)
- added Q22: 2N3904, Package_TO_SOT_THT:TO-92_Inline, F.Cu at (438.1, 450.2)
- added Q23: 2N3904, Package_TO_SOT_THT:TO-92_Inline, F.Cu at (438.1, 455.7)
- added Q24: 2N3904, Package_TO_SOT_THT:TO-92_Inline, F.Cu at (444.9, 450.2)
- added Q25: 2N3904, Package_TO_SOT_THT:TO-92_Inline, F.Cu at (585.6, 451.5)
- added Q26: 2N3904, Package_TO_SOT_THT:TO-92_Inline, F.Cu at (585.6, 457.0)
- added Q27: 2N3904, Package_TO_SOT_THT:TO-92_Inline, F.Cu at (592.5, 451.5)
- added Q28: 2N3904, Package_TO_SOT_THT:TO-92_Inline, F.Cu at (394.4, 451.1)
- added Q29: 2N3904, Package_TO_SOT_THT:TO-92_Inline, F.Cu at (394.4, 456.6)
- added Q30: 2N3904, Package_TO_SOT_THT:TO-92_Inline, F.Cu at (401.3, 451.1)
- added Q31: 2N3904, Package_TO_SOT_THT:TO-92_Inline, F.Cu at (522.0, 483.2)
- added Q32: 2N3904, Package_TO_SOT_THT:TO-92_Inline, F.Cu at (522.0, 488.7)
- added Q33: 2N3904, Package_TO_SOT_THT:TO-92_Inline, F.Cu at (528.9, 483.2)
- added Q34: 2N3904, Package_TO_SOT_THT:TO-92_Inline, F.Cu at (416.1, 484.0)
- added Q35: 2N3904, Package_TO_SOT_THT:TO-92_Inline, F.Cu at (416.1, 489.5)
- added Q36: 2N3904, Package_TO_SOT_THT:TO-92_Inline, F.Cu at (422.9, 484.0)
- added Q4: 2N3904, Package_TO_SOT_THT:TO-92_Inline, F.Cu at (509.1, 449.4)
- added Q5: 2N3904, Package_TO_SOT_THT:TO-92_Inline, F.Cu at (509.1, 454.9)
- added Q6: 2N3904, Package_TO_SOT_THT:TO-92_Inline, F.Cu at (516.0, 449.4)
- added Q7: 2N3904, Package_TO_SOT_THT:TO-92_Inline, F.Cu at (688.0, 414.5)
- added Q8: 2N3904, Package_TO_SOT_THT:TO-92_Inline, F.Cu at (688.0, 420.0)
- added Q9: 2N3904, Package_TO_SOT_THT:TO-92_Inline, F.Cu at (694.9, 414.5)
- added R10: 1000, Resistor_THT:R_Axial_DIN0207_L6.3mm_D2.5mm_P10.16mm_Horizontal, F.Cu at (679.8, 438.8)
- added R11: 1000, Resistor_THT:R_Axial_DIN0207_L6.3mm_D2.5mm_P10.16mm_Horizontal, F.Cu at (679.8, 451.2)
- added R12: 100, Resistor_THT:R_Axial_DIN0207_L6.3mm_D2.5mm_P10.16mm_Horizontal, F.Cu at (700.3, 434.2)
- added R13: 1000, Resistor_THT:R_Axial_DIN0207_L6.3mm_D2.5mm_P10.16mm_Horizontal, F.Cu at (611.3, 403.0)
- added R14: 1000, Resistor_THT:R_Axial_DIN0207_L6.3mm_D2.5mm_P10.16mm_Horizontal, F.Cu at (611.3, 415.4)
- added R15: 100, Resistor_THT:R_Axial_DIN0207_L6.3mm_D2.5mm_P10.16mm_Horizontal, F.Cu at (631.8, 398.4)
- added R16: 1000, Resistor_THT:R_Axial_DIN0207_L6.3mm_D2.5mm_P10.16mm_Horizontal, F.Cu at (420.1, 402.5)
- added R17: 1000, Resistor_THT:R_Axial_DIN0207_L6.3mm_D2.5mm_P10.16mm_Horizontal, F.Cu at (420.1, 415.0)
- added R18: 100, Resistor_THT:R_Axial_DIN0207_L6.3mm_D2.5mm_P10.16mm_Horizontal, F.Cu at (440.6, 398.0)
- added R19: 1000, Resistor_THT:R_Axial_DIN0207_L6.3mm_D2.5mm_P10.16mm_Horizontal, F.Cu at (608.8, 439.6)
- added R20: 1000, Resistor_THT:R_Axial_DIN0207_L6.3mm_D2.5mm_P10.16mm_Horizontal, F.Cu at (608.8, 452.1)
- added R21: 100, Resistor_THT:R_Axial_DIN0207_L6.3mm_D2.5mm_P10.16mm_Horizontal, F.Cu at (629.2, 435.1)
- added R22: 1000, Resistor_THT:R_Axial_DIN0207_L6.3mm_D2.5mm_P10.16mm_Horizontal, F.Cu at (417.6, 439.2)
- added R23: 1000, Resistor_THT:R_Axial_DIN0207_L6.3mm_D2.5mm_P10.16mm_Horizontal, F.Cu at (417.6, 451.6)
- added R24: 100, Resistor_THT:R_Axial_DIN0207_L6.3mm_D2.5mm_P10.16mm_Horizontal, F.Cu at (438.1, 434.6)
- added R25: 1000, Resistor_THT:R_Axial_DIN0207_L6.3mm_D2.5mm_P10.16mm_Horizontal, F.Cu at (565.2, 440.5)
- added R26: 1000, Resistor_THT:R_Axial_DIN0207_L6.3mm_D2.5mm_P10.16mm_Horizontal, F.Cu at (565.2, 452.9)
- added R27: 100, Resistor_THT:R_Axial_DIN0207_L6.3mm_D2.5mm_P10.16mm_Horizontal, F.Cu at (585.6, 435.9)
- added R28: 1000, Resistor_THT:R_Axial_DIN0207_L6.3mm_D2.5mm_P10.16mm_Horizontal, F.Cu at (374.0, 440.0)
- added R29: 1000, Resistor_THT:R_Axial_DIN0207_L6.3mm_D2.5mm_P10.16mm_Horizontal, F.Cu at (374.0, 452.5)
- added R30: 100, Resistor_THT:R_Axial_DIN0207_L6.3mm_D2.5mm_P10.16mm_Horizontal, F.Cu at (394.4, 435.5)
- added R31: 1000, Resistor_THT:R_Axial_DIN0207_L6.3mm_D2.5mm_P10.16mm_Horizontal, F.Cu at (501.5, 472.1)
- added R32: 1000, Resistor_THT:R_Axial_DIN0207_L6.3mm_D2.5mm_P10.16mm_Horizontal, F.Cu at (501.5, 484.6)
- added R33: 100, Resistor_THT:R_Axial_DIN0207_L6.3mm_D2.5mm_P10.16mm_Horizontal, F.Cu at (522.0, 467.6)
- added R34: 1000, Resistor_THT:R_Axial_DIN0207_L6.3mm_D2.5mm_P10.16mm_Horizontal, F.Cu at (395.6, 473.0)
- added R35: 1000, Resistor_THT:R_Axial_DIN0207_L6.3mm_D2.5mm_P10.16mm_Horizontal, F.Cu at (395.6, 485.4)
- added R36: 100, Resistor_THT:R_Axial_DIN0207_L6.3mm_D2.5mm_P10.16mm_Horizontal, F.Cu at (416.1, 468.4)
- added R4: 1000, Resistor_THT:R_Axial_DIN0207_L6.3mm_D2.5mm_P10.16mm_Horizontal, F.Cu at (488.7, 438.3)
- added R5: 1000, Resistor_THT:R_Axial_DIN0207_L6.3mm_D2.5mm_P10.16mm_Horizontal, F.Cu at (488.7, 450.8)
- added R6: 100, Resistor_THT:R_Axial_DIN0207_L6.3mm_D2.5mm_P10.16mm_Horizontal, F.Cu at (509.1, 433.8)
- added R7: 1000, Resistor_THT:R_Axial_DIN0207_L6.3mm_D2.5mm_P10.16mm_Horizontal, F.Cu at (667.5, 403.5)
- added R8: 1000, Resistor_THT:R_Axial_DIN0207_L6.3mm_D2.5mm_P10.16mm_Horizontal, F.Cu at (667.5, 415.9)
- added R9: 100, Resistor_THT:R_Axial_DIN0207_L6.3mm_D2.5mm_P10.16mm_Horizontal, F.Cu at (688.0, 398.9)
- added REF**: PinHeader_1x02_P2.54mm_Vertical, Connector_PinHeader_2.54mm:PinHeader_1x02_P2.54mm_Vertical, F.Cu at (335.0, 372.2)
- moved SW2 370.4 mm to (316.8, 484.5), turned to 90 degrees
- moved SW1 362.6 mm to (315.0, 417.2), turned to 90 degrees
- moved R2 276.8 mm to (476.3, 415.5)
- moved R1 276.6 mm to (476.3, 403.0)
- moved R3 256.2 mm to (496.8, 398.4), turned to -90 degrees
- moved Q1 250.3 mm to (496.8, 414.1), turned to 90 degrees
- moved Q2 250.3 mm to (496.8, 419.6), turned to 90 degrees
- moved Q3 243.1 mm to (503.7, 414.1), turned to 90 degrees
- moved D2 70.8 mm to (735.8, 446.2), turned to 180 degrees
- moved R38 64.6 mm to (736.0, 439.8), turned to 90 degrees
- moved D1 50.8 mm to (734.0, 408.5), turned to -90 degrees
- moved R37 48.7 mm to (734.0, 404.6), turned to 90 degrees
Connections:
- Q3 pad 1: /NAND11/C -> /Register/D-Flip-Flop/D-Latch/Q
- R1 pad 1: /NAND11/A -> /Register/D-Flip-Flop/D-Latch/NAND12/C
- R2 pad 1: /NAND11/B -> /Register/D-Flip-Flop/D-Latch/!Q
- SW1 pad 1: +5V -> VCC
- SW2 pad 1: +5V -> VCC
Routing:
- net VCC: track 0.00 -> 2261.7 mm
- net /Register/D-Flip-Flop/D-Latch/Enable: track 0.00 -> 240.4 mm, vias 0 -> 2
- net /Register/D-Flip-Flop/D-Latch/Q: track 0.00 -> 238.0 mm, vias 0 -> 2
- net /Register/D-Flip-Flop/Data: track 0.00 -> 194.3 mm, vias 0 -> 2
- net /Register/D-Flip-Flop/D-Latch1/Enable: track 0.00 -> 154.5 mm, vias 0 -> 2
- net /Register/D-Flip-Flop/!Q: track 0.00 -> 105.9 mm, vias 0 -> 1
- net /Register/D-Flip-Flop/Clock: track 0.00 -> 103.9 mm, vias 0 -> 1
- net /Register/D-Flip-Flop/D-Latch/!Q: track 0.00 -> 90.7 mm, vias 0 -> 1
- net /Register/D-Flip-Flop/Q: track 0.00 -> 84.8 mm, vias 0 -> 1
- net Net-(Q34-C): track 0.00 -> 61.8 mm
- net Net-(Q31-C): track 0.00 -> 61.8 mm
- net Net-(Q25-C): track 0.00 -> 61.8 mm
- net Net-(Q22-C): track 0.00 -> 61.8 mm
- net Net-(Q19-C): track 0.00 -> 61.8 mm
- net Net-(Q13-C): track 0.00 -> 61.8 mm
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- added copper zone on B.Cu, net GND
- added copper zone on F.Cu, net GND
Other:
- board outline added: 457.2 x 153.8 mm
- board text added: "+5v"
- board text added: "A"
- board text added: "B"
- board text added: "C"
- board text added: "Clock"
- board text added: "D - Flip Flop ------------------ 36 Transistors 38 Resistors"
- board text added: "D-Latch"
- board text added: "Data"
- board text added: "Enable"
- board text added: "GND"
- board text added: "NAND"
- board text added: "Q"
- board text added: "RESET"
- board text added: "SET"
- board text added: "SR-LATCH"
- board text added: "VCC"
- board text added: "_ Q"

Commit message: Added Some stuff
Parts:
- removed D1, D2: LED, LED_THT:LED_D5.0mm_Clear
- removed Q1, Q13, Q14, Q15, Q16, Q17, Q18, Q19, Q2, Q20, Q21, Q22, Q23, Q24, Q25, Q26, Q27, Q28, Q29, Q3, Q30, Q31, Q32, Q33, Q34, Q35, Q36, Q4, Q5, Q6, Q7, Q8, Q9: 2N3904, Package_TO_SOT_THT:TO-92_Inline
- removed R1, R13, R14, R16, R17, R19, R20, R22, R23, R25, R26, R28, R29, R31, R32, R34, R35, R37, R38, R4, R5, R7, R8: 1000, Resistor_THT:R_Axial_DIN0207_L6.3mm_D2.5mm_P10.16mm_Horizontal
- removed R15, R18, R21, R24, R27, R3, R30, R33, R36, R6, R9: 100, Resistor_THT:R_Axial_DIN0207_L6.3mm_D2.5mm_P10.16mm_Horizontal
- removed REF**: PinHeader_1x02_P2.54mm_Vertical, Connector_PinHeader_2.54mm:PinHeader_1x02_P2.54mm_Vertical
- removed SW1, SW2: SW_Push_Dual, Button_Switch_THT:SW_PUSH_6mm
- added D3: LED, LED_THT:LED_D5.0mm_Clear, F.Cu at (722.2, 445.8)
- added SW4: SW_Push_Dual, Button_Switch_THT:SW_PUSH_6mm, F.Cu at (666.2, 434.5)
- added SW6: SW_Push_Dual, Button_Switch_THT:SW_PUSH_6mm, F.Cu at (665.8, 451.5)
- moved R2 251.2 mm to (725.7, 446.0)
Connections:
- Q12 pad 1: /Register/D-Flip-Flop/!Q -> /Register/D-Flip-Flop/D-Latch1/SR-Latch/NAND11/C
- R10 pad 1: /Register/D-Flip-Flop/Q -> /Register/D-Flip-Flop/D-Latch1/SR-Latch/NAND11/A
- R11 pad 1: /Register/D-Flip-Flop/D-Latch1/NAND13/C -> /Register/D-Flip-Flop/D-Latch1/SR-Latch/NAND11/B
- R2 pad 1: /Register/D-Flip-Flop/D-Latch/!Q -> Net-(D3-K)
- R2 pad 2: Net-(Q2-B) -> GND
Routing:
- net VCC: track 2261.7 -> 175.7 mm
- net /Register/D-Flip-Flop/D-Latch/Enable: track 240.4 -> 0.00 mm, vias 2 -> 0
- net /Register/D-Flip-Flop/D-Latch/Q: track 238.0 -> 0.00 mm, vias 2 -> 0
- net /Register/D-Flip-Flop/Data: track 194.3 -> 0.00 mm, vias 2 -> 0
- net /Register/D-Flip-Flop/D-Latch1/Enable: track 154.5 -> 0.00 mm, vias 2 -> 0
- net /Register/D-Flip-Flop/!Q: track 105.9 -> 0.00 mm, vias 1 -> 0
- net /Register/D-Flip-Flop/Clock: track 103.9 -> 0.00 mm, vias 1 -> 0
- net /Register/D-Flip-Flop/D-Latch/!Q: track 90.7 -> 0.00 mm, vias 1 -> 0
- net /Register/D-Flip-Flop/Q: track 84.8 -> 0.00 mm, vias 1 -> 0
- net Net-(Q34-C): track 61.8 -> 0.00 mm
- net Net-(Q31-C): track 61.8 -> 0.00 mm
- net Net-(Q25-C): track 61.8 -> 0.00 mm
- net Net-(Q22-C): track 61.8 -> 0.00 mm
- net Net-(Q19-C): track 61.8 -> 0.00 mm
- net Net-(Q13-C): track 61.8 -> 0.00 mm
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Other:
- board size 457.2 x 153.8 mm -> 79.2 x 32.8 mm
- board text added: "NAND GATE A | B | C ------ 0 | 0 | 1 0 | 1 | 1 1 | 0 | 1 1 | 1 | 0"
- board text removed: "+5v"
- board text removed: "Clock"
- board text removed: "D - Flip Flop ------------------ 36 Transistors 38 Resistors"
- board text removed: "D-Latch"
- board text removed: "Data"
- board text removed: "Enable"
- board text removed: "Q"
- board text removed: "RESET"
- board text removed: "SET"
- board text removed: "SR-LATCH"
- board text removed: "_ Q"
