File: Sandbox/nand.kicad_sch (KiCad schematic)
At the start: 6 parts, among them Q1 2N3904, Q2 2N3904, Q3 2N3904

Commit message: Test D-Latch Finished
Parts:
- renumbered R2 to R1, R3 to R2, R1 to R3
