File: Sandbox/nand_gate/D-Latch.kicad_sch (KiCad schematic)
At the start: 0 parts

Commit message: D-Latch Done
Other:
- added sheet nand_gate2 (nand__gate.kicad_sch)
- added sheet nand_gate3 (nand__gate.kicad_sch)
- added sheet nand_gate4 (nand__gate.kicad_sch)
- sheet SR-Latch ports: added !Q, Q, Reset, Set; removed none
Changed lines of the file:
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@@
 (kicad_sch (version 20230121) (generator eeschema)
   (paper "A4")
-  (sheet (at 91.44 58.42) (size 35.56 19.05) (fields_autoplaced)
+  (junction (at 57.15 73.66) (diameter 0) (color 0 0 0 0)
+  )
+  (wire (pts (xy 73.66 76.2) (xy 82.55 76.2))
+    (stroke (width 0) (type default))
+  )
+  (wire (pts (xy 57.15 73.66) (xy 57.15 59.69))
+    (stroke (width 0) (type default))
+  )
+  (wire (pts (xy 129.54 73.66) (xy 133.35 73.66))
+    (stroke (width 0) (type default))
+  )
+  (wire (pts (xy 57.15 80.01) (xy 60.96 80.01))
+    (stroke (width 0) (type default))
+  )
+  (wire (pts (xy 57.15 59.69) (xy 87.63 59.69))
+    (stroke (width 0) (type default))
+  )
+  (wire (pts (xy 60.96 73.66) (xy 57.15 73.66))
+    (stroke (width 0) (type default))
+  )
+  (wire (pts (xy 80.01 73.66) (xy 87.63 73.66))
+    (stroke (width 0) (type default))
+  )
+  (wire (pts (xy 100.33 76.2) (xy 106.68 76.2))
+    (stroke (width 0) (type default))
+  )
+  (wire (pts (xy 82.55 80.01) (xy 87.63 80.01))
+    (stroke (width 0) (type default))
+  )
+  (wire (pts (xy 57.15 73.66) (xy 57.15 80.01))
+    (stroke (width 0) (type default))
+  )
+  (wire (pts (xy 106.68 76.2) (xy 106.68 73.66))
+    (stroke (width 0) (type default))
+  )
+  (wire (pts (xy 100.33 62.23) (xy 111.76 62.23))
+    (stroke (width 0) (type default))
+  )
+  (wire (pts (xy 82.55 76.2) (xy 82.55 80.01))
+    (stroke (width 0) (type default))
+  )
+  (wire (pts (xy 80.01 66.04) (xy 87.63 66.04))
+    (stroke (width 0) (type default))
+  )
+  (wire (pts (xy 80.01 66.04) (xy 80.01 73.66))
+    (stroke (width 0) (type default))
+  )
+  (wire (pts (xy 129.54 62.23) (xy 133.35 62.23))
+    (stroke (width 0) (type default))
+  )
+  (wire (pts (xy 106.68 73.66) (xy 111.76 73.66))
+    (stroke (width 0) (type default))
+  )
+  (hierarchical_label "!Q" (shape input) (at 133.35 73.66 0) (fields_autoplaced)
+    (effects (font (size 1.27 1.27)) (justify left))
+  )
+  (hierarchical_label "Q" (shape input) (at 133.35 62.23 0) (fields_autoplaced)
+    (effects (font (size 1.27 1.27)) (justify left))
+  )
+  (hierarchical_label "Data" (shape input) (at 57.15 63.5 180) (fields_autoplaced)
+    (effects (font (size 1.27 1.27)) (justify right))
+  )
+  (hierarchical_label "Enable" (shape input) (at 80.01 67.31 180) (fields_autoplaced)
+    (effects (font (size 1.27 1.27)) (justify right))
+  )
+  (sheet (at 111.76 60.96) (size 17.78 13.97) (fields_autoplaced)
     (stroke (width 0.1524) (type solid))
     (fill (color 0 0 0 0.0000))
-    (property "Sheetname" "SR-Latch" (at 91.44 57.7084 0)
+    (property "Sheetname" "SR-Latch" (at 111.76 60.2484 0)
       (effects (font (size 1.27 1.27)) (justify left bottom))
     )
-    (property "Sheetfile" "SR_LATCH.kicad_sch" (at 91.44 78.0546 0)
+    (property "Sheetfile" "SR_LATCH.kicad_sch" (at 111.76 75.5146 0)
       (effects (font (size 1.27 1.27)) (justify left top))
+    )
+    (pin "Reset" input (at 111.76 73.66 180)
+      (effects (font (size 1.27 1.27)) (justify left))
+    )
+    (pin "Q" input (at 129.54 62.23 0)
+      (effects (font (size 1.27 1.27)) (justify right))
+    )
+    (pin "Set" input (at 111.76 62.23 180)
+      (effects (font (size 1.27 1.27)) (justify left))
+    )
+    (pin "!Q" input (at 129.54 73.66 0)
+      (effects (font (size 1.27 1.27)) (justify right))
     )
     (instances
@@
       )
     )
+  )
+  (sheet (at 87.63 72.39) (size 12.7 8.89)
+    (stroke (width 0.1524) (type solid))
+    (fill (color 0 0 0 0.0000))
+    (property "Sheetname" "nand_gate3" (at 87.63 71.6784 0)
+      (effects (font (size 1.27 1.27)) (justify left bottom))
+    )
+    (property "Sheetfile" "nand__gate.kicad_sch" (at 82.55 81.28 0)
+      (effects (font (size 1.27 1.27)) (justify left top))
+    )
+    (pin "B" input (at 87.63 80.01 180)
+      (effects (font (size 1.27 1.27)) (justify left))
+    )
+    (pin "A" input (at 87.63 73.66 180)
+      (effects (font (size 1.27 1.27)) (justify left))
+    )
+    (pin "C" input (at 100.33 76.2 0)
+      (effects (font (size 1.27 1.27)) (justify right))
+    )
+    (instances
+      (project "nand_gate"
+        (path "/ae45e9d9-ebb5-4d6c-8dad-99eadd2be5c5/2e87dc14-878c-467c-8594-4a57b58f886f/6b230bbb-3b41-4fd2-a79b-e0cf50894ec7/0ad4044b-a9cd-452a-a5d6-d186c7bbd4c9" (page "5"))
+        (path "/ae45e9d9-ebb5-4d6c-8dad-99eadd2be5c5/2e87dc14-878c-467c-8594-4a57b58f886f/6b230bbb-3b41-4fd2-a79b-e0cf50894ec7" (page "8"))
+      )
+    )
+  )
+  (sheet (at 60.96 72.39) (size 12.7 8.89)
+    (stroke (width 0.1524) (type solid))
+    (fill (color 0 0 0 0.0000))
+    (property "Sheetname" "nand_gate4" (at 60.96 71.6784 0)
+      (effects (font (size 1.27 1.27)) (justify left bottom))
+    )
+    (property "Sheetfile" "nand__gate.kicad_sch" (at 55.88 81.28 0)
+      (effects (font (size 1.27 1.27)) (justify left top))
+    )
+    (pin "B" input (at 60.96 80.01 180)
+      (effects (font (size 1.27 1.27)) (justify left))
+    )
+    (pin "A" input (at 60.96 73.66 180)
+      (effects (font (size 1.27 1.27)) (justify left))
+    )
+    (pin "C" input (at 73.66 76.2 0)
+      (effects (font (size 1.27 1.27)) (justify right))
+    )
+    (instances
+      (project "nand_gate"
+        (path "/ae45e9d9-ebb5-4d6c-8dad-99eadd2be5c5/2e87dc14-878c-467c-8594-4a57b58f886f/6b230bbb-3b41-4fd2-a79b-e0cf50894ec7/0ad4044b-a9cd-452a-a5d6-d186c7bbd4c9" (page "5"))
+        (path "/ae45e9d9-ebb5-4d6c-8dad-99eadd2be5c5/2e87dc14-878c-467c-8594-4a57b58f886f/6b230bbb-3b41-4fd2-a79b-e0cf50894ec7" (page "9"))
+      )
+    )
+  )
+  (sheet (at 87.63 58.42) (size 12.7 8.89)
+    (stroke (width 0.1524) (type solid))
+    (fill (color 0 0 0 0.0000))
+    (property "Sheetname" "nand_gate2" (at 87.63 57.7084 0)
+      (effects (font (size 1.27 1.27)) (justify left bottom))
+    )
+    (property "Sheetfile" "nand__gate.kicad_sch" (at 82.55 54.61 0)
+      (effects (font (size 1.27 1.27)) (justify left top))
+    )
+    (pin "B" input (at 87.63 66.04 180)
+      (effects (font (size 1.27 1.27)) (justify left))
+    )
+    (pin "A" input (at 87.63 59.69 180)
+      (effects (font (size 1.27 1.27)) (justify left))
+    )
+    (pin "C" input (at 100.33 62.23 0)
+      (effects (font (size 1.27 1.27)) (justify right))
+    )
+    (instances
+      (project "nand_gate"
+        (path "/ae45e9d9-ebb5-4d6c-8dad-99eadd2be5c5/2e87dc14-878c-467c-8594-4a57b58f886f/6b230bbb-3b41-4fd2-a79b-e0cf50894ec7/0ad4044b-a9cd-452a-a5d6-d186c7bbd4c9" (page "5"))
+        (path "/ae45e9d9-ebb5-4d6c-8dad-99eadd2be5c5/2e87dc14-878c-467c-8594-4a57b58f886f/6b230bbb-3b41-4fd2-a79b-e0cf50894ec7" (page "7"))
+      )
+    )
