File: Sandbox/nand_gate/SR_LATCH.kicad_sch (KiCad schematic)
At the start: 0 parts

Commit message: Updating schematic
Other:
- sheet nand_gate ports: added A, B, C; removed none
Changed lines of the file:
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@@
 (kicad_sch (version 20230121) (generator eeschema)
   (paper "A4")
-  (sheet (at 66.04 49.53) (size 46.99 33.02) (fields_autoplaced)
+  (sheet (at 128.27 77.47) (size 12.7 8.89) (fields_autoplaced)
     (stroke (width 0.1524) (type solid))
     (fill (color 0 0 0 0.0000))
-    (property "Sheetname" "nand_gate" (at 66.04 48.8184 0)
+    (property "Sheetname" "nand_gate" (at 128.27 76.7584 0)
       (effects (font (size 1.27 1.27)) (justify left bottom))
     )
-    (property "Sheetfile" "nand__gate.kicad_sch" (at 66.04 83.1346 0)
+    (property "Sheetfile" "nand__gate.kicad_sch" (at 128.27 86.9446 0)
       (effects (font (size 1.27 1.27)) (justify left top))
     )
+    (pin "B" input (at 128.27 85.09 180)
+      (effects (font (size 1.27 1.27)) (justify left))
+    )
+    (pin "A" input (at 128.27 78.74 180)
+      (effects (font (size 1.27 1.27)) (justify left))
+    )
+    (pin "C" input (at 140.97 81.28 0)
+      (effects (font (size 1.27 1.27)) (justify right))
+    )
     (instances

Commit message: D-Latch Done
Other:
- added sheet nand_gate1 (nand__gate.kicad_sch)
Changed lines of the file:
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@@
 (kicad_sch (version 20230121) (generator eeschema)
   (paper "A4")
+  (junction (at 142.24 104.14) (diameter 0) (color 0 0 0 0)
+  )
+  (junction (at 142.24 81.28) (diameter 0) (color 0 0 0 0)
+  )
+  (wire (pts (xy 140.97 104.14) (xy 142.24 104.14))
+    (stroke (width 0) (type default))
+  )
+  (wire (pts (xy 123.19 85.09) (xy 128.27 85.09))
+    (stroke (width 0) (type default))
+  )
+  (wire (pts (xy 142.24 104.14) (xy 148.59 104.14))
+    (stroke (width 0) (type default))
+  )
+  (wire (pts (xy 127 101.6) (xy 128.27 101.6))
+    (stroke (width 0) (type default))
+  )
+  (wire (pts (xy 123.19 97.79) (xy 123.19 85.09))
+    (stroke (width 0) (type default))
+  )
+  (wire (pts (xy 142.24 104.14) (xy 142.24 97.79))
+    (stroke (width 0) (type default))
+  )
+  (wire (pts (xy 124.46 107.95) (xy 128.27 107.95))
+    (stroke (width 0) (type default))
+  )
+  (wire (pts (xy 140.97 81.28) (xy 142.24 81.28))
+    (stroke (width 0) (type default))
+  )
+  (wire (pts (xy 142.24 97.79) (xy 123.19 97.79))
+    (stroke (width 0) (type default))
+  )
+  (wire (pts (xy 142.24 81.28) (xy 142.24 95.25))
+    (stroke (width 0) (type default))
+  )
+  (wire (pts (xy 142.24 81.28) (xy 146.05 81.28))
+    (stroke (width 0) (type default))
+  )
+  (wire (pts (xy 127 95.25) (xy 127 101.6))
+    (stroke (width 0) (type default))
+  )
+  (wire (pts (xy 142.24 95.25) (xy 127 95.25))
+    (stroke (width 0) (type default))
+  )
+  (wire (pts (xy 124.46 78.74) (xy 128.27 78.74))
+    (stroke (width 0) (type default))
+  )
+  (hierarchical_label "Q" (shape input) (at 146.05 81.28 0) (fields_autoplaced)
+    (effects (font (size 1.27 1.27)) (justify left))
+  )
+  (hierarchical_label "Set" (shape input) (at 124.46 78.74 180) (fields_autoplaced)
+    (effects (font (size 1.27 1.27)) (justify right))
+  )
+  (hierarchical_label "!Q" (shape input) (at 148.59 104.14 0) (fields_autoplaced)
+    (effects (font (size 1.27 1.27)) (justify left))
+  )
+  (hierarchical_label "Reset" (shape input) (at 124.46 107.95 180) (fields_autoplaced)
+    (effects (font (size 1.27 1.27)) (justify right))
+  )
   (sheet (at 128.27 77.47) (size 12.7 8.89) (fields_autoplaced)
     (stroke (width 0.1524) (type solid))
@@
       )
     )
+  )
+  (sheet (at 128.27 100.33) (size 12.7 8.89) (fields_autoplaced)
+    (stroke (width 0.1524) (type solid))
+    (fill (color 0 0 0 0.0000))
+    (property "Sheetname" "nand_gate1" (at 128.27 99.6184 0)
+      (effects (font (size 1.27 1.27)) (justify left bottom))
+    )
+    (property "Sheetfile" "nand__gate.kicad_sch" (at 128.27 109.8046 0)
+      (effects (font (size 1.27 1.27)) (justify left top))
+    )
+    (pin "B" input (at 128.27 107.95 180)
+      (effects (font (size 1.27 1.27)) (justify left))
+    )
+    (pin "A" input (at 128.27 101.6 180)
+      (effects (font (size 1.27 1.27)) (justify left))
+    )
+    (pin "C" input (at 140.97 104.14 0)
+      (effects (font (size 1.27 1.27)) (justify right))
+    )
+    (instances
+      (project "nand_gate"
+        (path "/ae45e9d9-ebb5-4d6c-8dad-99eadd2be5c5/2e87dc14-878c-467c-8594-4a57b58f886f/6b230bbb-3b41-4fd2-a79b-e0cf50894ec7/0ad4044b-a9cd-452a-a5d6-d186c7bbd4c9" (page "6"))
+      )
+    )
