File: Sandbox/nand_gate/nand__gate.kicad_sch (KiCad schematic)
At the start: 8 parts, among them Q1 2N3904, Q2 2N3904, Q3 2N3904

Commit message: Moved Some Things Around
Parts:
- removed D1: LED, LED_THT:LED_D5.0mm, symbol Device:LED
- removed Q1, Q2, Q3: 2N3904, Package_TO_SOT_THT:TO-92_Inline, symbol Transistor_BJT:2N3904
- removed R4: 150, Resistor_THT:R_Axial_DIN0207_L6.3mm_D2.5mm_P7.62mm_Horizontal, symbol Device:R
- added Q12, Q24, Q48: Q_NPN_BEC, Package_TO_SOT_SMD:SOT-23, symbol Device:Q_NPN_BEC
- R1, R2, R3: footprint Resistor_THT:R_Axial_DIN0207_L6.3mm_D2.5mm_P7.62mm_Horizontal -> Resistor_SMD:R_0402_1005Metric
Connections:
- net C: now also Q48.2 (E)
- net GND: now also Q24.2 (E)
- net VCC: now also Q48.3 (C)
- net at R1.2: now also Q12.1 (B)
- net at R3.1: now also Q12.3 (C), Q48.1 (B)
- net at R2.2: now also Q24.1 (B)
- new net: Q12.2 (E), Q24.3 (C)
Other:
- moved on the sheet: R3
