File: Sandbox/nand_gate/nand_gate.kicad_pcb (KiCad board)
At the start: 2 copper layers, 96 parts, among them Q1 2N3904, Q10 2N3904, Q11 2N3904, Q12 2N3904, Q13 2N3904, Q14 2N3904, Q15 2N3904, Q16 2N3904, Q17 2N3904, Q18 2N3904, Q19 2N3904, Q2 2N3904, Q20 2N3904, Q21 2N3904, Q22 2N3904, Q23 2N3904, Q24 2N3904, Q25 2N3904, Q26 2N3904, Q27 2N3904, Q28 2N3904, Q29 2N3904, Q3 2N3904, Q30 2N3904, Q31 2N3904, Q32 2N3904, Q33 2N3904, Q34 2N3904, Q35 2N3904, Q36 2N3904, Q4 2N3904, Q5 2N3904, Q6 2N3904, Q7 2N3904, Q8 2N3904, Q9 2N3904

Commit message: Moved Some Things Around
Parts:
- removed D1, D10, D11, D12, D2, D3, D4, D5, D6, D7, D8, D9: LED, LED_THT:LED_D5.0mm
- removed Q28, Q29, Q30, Q31, Q32, Q33, Q34, Q35, Q36: 2N3904, Package_TO_SOT_THT:TO-92_Inline
- removed R16, R20, R24, R28, R32, R36, R40, R44, R48: 150, Resistor_THT:R_Axial_DIN0207_L6.3mm_D2.5mm_P7.62mm_Horizontal
- added Q37: Q_NPN_BEC, Package_TO_SOT_SMD:SOT-23, F.Cu at (218.1, 68.0)
- added Q38: Q_NPN_BEC, Package_TO_SOT_SMD:SOT-23, F.Cu at (218.1, 83.3)
- added Q39: Q_NPN_BEC, Package_TO_SOT_SMD:SOT-23, F.Cu at (247.5, 52.6)
- added Q40: Q_NPN_BEC, Package_TO_SOT_SMD:SOT-23, F.Cu at (227.9, 52.6)
- added Q41: Q_NPN_BEC, Package_TO_SOT_SMD:SOT-23, F.Cu at (237.7, 52.6)
- added Q42: Q_NPN_BEC, Package_TO_SOT_SMD:SOT-23, F.Cu at (237.7, 83.3)
- added Q43: Q_NPN_BEC, Package_TO_SOT_SMD:SOT-23, F.Cu at (247.5, 68.0)
- added Q44: Q_NPN_BEC, Package_TO_SOT_SMD:SOT-23, F.Cu at (227.9, 68.0)
- added Q45: Q_NPN_BEC, Package_TO_SOT_SMD:SOT-23, F.Cu at (237.7, 68.0)
- added Q46: Q_NPN_BEC, Package_TO_SOT_SMD:SOT-23, F.Cu at (227.9, 83.3)
- added Q47: Q_NPN_BEC, Package_TO_SOT_SMD:SOT-23, F.Cu at (257.3, 52.6)
- added Q48: Q_NPN_BEC, Package_TO_SOT_SMD:SOT-23, F.Cu at (218.1, 52.6)
- Q1, Q10, Q11, Q12, Q13, Q14, Q15, Q16, Q17, Q18, Q19, Q2, Q20, Q21, Q22, Q23, Q24, Q25, Q26, Q27, Q3, Q4, Q5, Q6, Q7, Q8, Q9: value 2N3904 -> Q_NPN_BEC; footprint Package_TO_SOT_THT:TO-92_Inline -> Package_TO_SOT_SMD:SOT-23
- R1, R10, R11, R13, R14, R15, R17, R18, R19, R2, R21, R22, R23, R25, R26, R27, R29, R3, R30, R31, R33, R34, R35, R37, R38, R39, R41, R42, R43, R45, R46, R47, R5, R6, R7, R9: footprint Resistor_THT:R_Axial_DIN0207_L6.3mm_D2.5mm_P7.62mm_Horizontal -> Resistor_SMD:R_0402_1005Metric
- R12, R4, R8: value 150 -> 1k; footprint Resistor_THT:R_Axial_DIN0207_L6.3mm_D2.5mm_P7.62mm_Horizontal -> Resistor_SMD:R_0402_1005Metric
- moved Q7 213.9 mm to (247.5, 59.1), turned to 0 degrees
- moved R11 211.4 mm to (251.4, 46.5)
- moved Q11 210.3 mm to (257.3, 43.8), turned to 0 degrees
- moved R9 204.1 mm to (251.4, 42.5), turned to 0 degrees
- moved R10 203.9 mm to (251.4, 44.5), turned to 0 degrees
- moved Q9 203.0 mm to (237.7, 59.1), turned to 0 degrees
- moved R13 198.4 mm to (231.8, 42.5)
- moved R14 197.7 mm to (231.8, 44.5)
- moved Q8 193.8 mm to (227.9, 59.1), turned to 0 degrees
- moved R15 189.5 mm to (231.8, 46.5), turned to 0 degrees
- moved Q6 183.3 mm to (237.7, 74.5), turned to 0 degrees
- moved Q5 180.8 mm to (237.7, 43.8), turned to 0 degrees
- moved Q10 180.4 mm to (227.9, 74.5), turned to 0 degrees
- moved Q3 180.0 mm to (247.5, 43.8), turned to 0 degrees
- moved Q4 171.3 mm to (227.9, 43.8), turned to 0 degrees
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Connections:
- Q1 pad 1: Net-(Q1-E) -> Net-(Q1-B)
- Q1 pad 2: Net-(Q1-B) -> Net-(Q1-E)
- Q10 pad 1: Net-(Q10-E) -> Net-(Q10-B)
- Q10 pad 2: Net-(Q10-B) -> Net-(Q10-E)
- Q11 pad 1: GND -> Net-(Q11-B)
- Q11 pad 2: Net-(Q11-B) -> Net-(Q11-E)
- Q11 pad 3: Net-(Q10-E) -> Net-(Q11-C)
- Q12 pad 1: Net-(Q12-E) -> Net-(Q12-B)
- Q12 pad 2: Net-(Q10-C) -> Net-(Q12-E)
- Q12 pad 3: VCC -> Net-(Q12-C)
- Q13 pad 1: Net-(Q13-E) -> Net-(Q13-B)
- Q13 pad 2: Net-(Q13-B) -> GND
- Q13 pad 3: Net-(Q13-C) -> Net-(Q1-E)
- Q14 pad 1: GND -> Net-(Q14-B)
- Q14 pad 2: Net-(Q14-B) -> GND
- Q14 pad 3: Net-(Q13-E) -> Net-(Q14-C)
- Q15 pad 1: Net-(Q15-E) -> Net-(Q15-B)
- Q15 pad 2: Net-(Q13-C) -> GND
- Q15 pad 3: VCC -> Net-(Q15-C)
- Q16 pad 1: Net-(Q16-E) -> Net-(Q16-B)
- Q16 pad 2: Net-(Q16-B) -> GND
- Q17 pad 1: GND -> Net-(Q17-B)
- Q17 pad 2: Net-(Q17-B) -> GND
- Q17 pad 3: Net-(Q16-E) -> Net-(Q17-C)
- Q18 pad 1: Net-(Q18-E) -> Net-(Q18-B)
- Q18 pad 2: Net-(Q16-C) -> GND
- Q18 pad 3: VCC -> Net-(Q18-C)
- Q19 pad 1: Net-(Q19-E) -> Net-(Q19-B)
- Q19 pad 2: Net-(Q19-B) -> GND
- Q2 pad 1: GND -> Net-(Q2-B)
- Q2 pad 2: Net-(Q2-B) -> Net-(Q14-C)
- Q2 pad 3: Net-(Q1-E) -> Net-(Q2-C)
- Q20 pad 1: GND -> Net-(Q20-B)
- Q20 pad 2: Net-(Q20-B) -> GND
- Q20 pad 3: Net-(Q19-E) -> Net-(Q20-C)
- Q21 pad 1: Net-(Q21-E) -> Net-(Q21-B)
- Q21 pad 2: Net-(Q19-C) -> GND
- Q21 pad 3: VCC -> Net-(Q21-C)
- Q22 pad 1: Net-(Q22-E) -> Net-(Q22-B)
- Q22 pad 2: Net-(Q22-B) -> GND
- Q22 pad 3: Net-(Q22-C) -> Net-(Q10-E)
- Q23 pad 1: GND -> Net-(Q23-B)
- Q23 pad 2: Net-(Q23-B) -> GND
- Q23 pad 3: Net-(Q22-E) -> Net-(Q11-E)
- Q24 pad 1: Net-(Q24-E) -> Net-(Q24-B)
- Q24 pad 2: Net-(Q22-C) -> GND
- Q24 pad 3: VCC -> Net-(Q12-E)
- Q25 pad 1: Net-(Q25-E) -> Net-(Q25-B)
- Q25 pad 2: Net-(Q25-B) -> Net-(Q25-E)
- Q26 pad 1: GND -> Net-(Q26-B)
- Q26 pad 2: Net-(Q26-B) -> GND
- Q27 pad 1: Net-(Q27-E) -> Net-(Q25-C)
- Q27 pad 2: Net-(Q25-C) -> /nand_gate7/C
- Q3 pad 1: Net-(Q3-E) -> Net-(Q3-B)
- Q3 pad 2: Net-(Q1-C) -> Net-(Q15-C)
- Q3 pad 3: VCC -> Net-(Q3-C)
- Q4 pad 1: Net-(Q4-E) -> Net-(Q4-B)
- Q4 pad 2: Net-(Q4-B) -> Net-(Q16-C)
- Q5 pad 1: GND -> Net-(Q5-B)
- Q5 pad 2: Net-(Q5-B) -> Net-(Q17-C)
- Q5 pad 3: Net-(Q4-E) -> Net-(Q41-B)
- Q6 pad 1: Net-(Q6-E) -> Net-(Q6-B)
- Q6 pad 2: Net-(Q4-C) -> Net-(Q18-C)
- Q6 pad 3: VCC -> Net-(Q42-B)
- Q7 pad 1: Net-(Q7-E) -> Net-(Q7-B)
- Q7 pad 2: Net-(Q7-B) -> Net-(Q19-C)
- Q7 pad 3: Net-(Q7-C) -> Net-(Q43-B)
- Q8 pad 1: GND -> Net-(Q8-B)
- Q8 pad 2: Net-(Q8-B) -> Net-(Q20-C)
- Q8 pad 3: Net-(Q7-E) -> Net-(Q44-B)
- Q9 pad 1: Net-(Q9-E) -> Net-(Q9-B)
- Q9 pad 2: Net-(Q7-C) -> Net-(Q21-C)
- Q9 pad 3: VCC -> Net-(Q45-B)
- R1 pad 2: Net-(Q1-B) -> Net-(Q2-B)
- R10 pad 2: Net-(Q8-B) -> Net-(Q15-B)
- R11 pad 1: Net-(Q7-C) -> Net-(Q3-C)
- R12 pad 1: Net-(Q9-E) -> Net-(Q25-C)
- R12 pad 2: /D-Flip Flop/D-Latch/SR-Latch/Set -> VCC
- R13 pad 2: Net-(Q10-B) -> Net-(Q4-B)
- R14 pad 2: Net-(Q11-B) -> Net-(Q16-B)
- R15 pad 1: Net-(Q10-C) -> Net-(Q4-C)
- R17 pad 2: Net-(Q13-B) -> Net-(Q5-B)
- R18 pad 2: Net-(Q14-B) -> Net-(Q17-B)
- R19 pad 1: Net-(Q13-C) -> Net-(Q41-B)
- R2 pad 2: Net-(Q2-B) -> Net-(Q14-B)
- R21 pad 2: Net-(Q16-B) -> Net-(Q6-B)
- R22 pad 2: Net-(Q17-B) -> Net-(Q18-B)
- R23 pad 1: Net-(Q16-C) -> Net-(Q42-B)
- R25 pad 2: Net-(Q19-B) -> Net-(Q7-B)
- R26 pad 2: Net-(Q20-B) -> Net-(Q19-B)
- R27 pad 1: Net-(Q19-C) -> Net-(Q43-B)
- R29 pad 2: Net-(Q22-B) -> Net-(Q8-B)
- R3 pad 1: Net-(Q1-C) -> Net-(Q2-C)
- R30 pad 2: Net-(Q23-B) -> Net-(Q20-B)
- R31 pad 1: Net-(Q22-C) -> Net-(Q44-B)
- R33 pad 2: Net-(Q25-B) -> Net-(Q9-B)
- R34 pad 2: Net-(Q26-B) -> Net-(Q21-B)
- R35 pad 1: Net-(Q25-C) -> Net-(Q45-B)
- R37 pad 2: Net-(Q28-B) -> Net-(Q10-B)
- R38 pad 2: Net-(Q29-B) -> Net-(Q22-B)
- R39 pad 1: Net-(Q28-C) -> Net-(Q10-C)
- R4 pad 1: Net-(Q3-E) -> /nand_gate7/A
- R4 pad 2: /D-Flip Flop/D-Latch/!Q -> Net-(Q25-B)
- R41 pad 2: Net-(Q31-B) -> Net-(Q11-B)
- R42 pad 2: Net-(Q32-B) -> Net-(Q23-B)
- R43 pad 1: Net-(Q31-C) -> Net-(Q11-C)
- R45 pad 2: Net-(Q34-B) -> Net-(Q12-B)
- R46 pad 2: Net-(Q35-B) -> Net-(Q24-B)
- R47 pad 1: Net-(Q34-C) -> Net-(Q12-C)
- R5 pad 2: Net-(Q4-B) -> Net-(Q1-B)
- R6 pad 2: Net-(Q5-B) -> Net-(Q13-B)
- R7 pad 1: Net-(Q4-C) -> Net-(Q1-C)
- R8 pad 1: Net-(Q6-E) -> /nand_gate7/B
- R8 pad 2: /D-Flip Flop/D-Latch/Q -> Net-(Q26-B)
- R9 pad 2: Net-(Q7-B) -> Net-(Q3-B)
Routing:
- net VCC: track 257.1 -> 5.90 mm
- net /D-Flip Flop/D-Latch/nand_gate3/B: track 123.7 -> 0.00 mm
- net /D-Flip Flop/D-Latch1/nand_gate3/B: track 123.7 -> 0.00 mm
- net /D-Flip Flop/D-Latch/Q: track 89.8 -> 0.00 mm
- net /D-Flip Flop/Data: track 59.6 -> 0.00 mm
- net /D-Flip Flop/D-Latch/Enable: track 47.8 -> 0.00 mm
- net /D-Flip Flop/D-Latch1/Enable: track 47.8 -> 0.00 mm
- net /D-Flip Flop/D-Latch/SR-Latch/Set: track 36.0 -> 0.00 mm
- net /D-Flip Flop/D-Latch1/SR-Latch/Set: track 36.0 -> 0.00 mm
- net /D-Flip Flop/D-Latch/SR-Latch/Reset: track 32.3 -> 0.00 mm
- net /D-Flip Flop/D-Latch1/SR-Latch/Reset: track 32.3 -> 0.00 mm
- net /D-Flip Flop/!Q: track 31.4 -> 0.00 mm
- net /D-Flip Flop/D-Latch/!Q: track 31.4 -> 0.00 mm
- net /D-Flip Flop/Q: track 30.2 -> 0.00 mm
- net Net-(Q34-C): track 18.2 -> 0.00 mm
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- added copper zone on B.Cu, net GND
- added copper zone on In1.Cu, net VCC
Other:
- board outline added: 94.8 x 91.8 mm
- copper layers 2 -> 4

Commit message: woring on layout.
Parts:
- added Q28: Q_NPN_BEC, Package_TO_SOT_SMD:SOT-23, F.Cu at (180.8, 30.7)
- added Q29: Q_NPN_BEC, Package_TO_SOT_SMD:SOT-23, F.Cu at (185.2, 30.7)
- added Q30: Q_NPN_BEC, Package_TO_SOT_SMD:SOT-23, F.Cu at (180.6, 27.0)
- added Q31: Q_NPN_BEC, Package_TO_SOT_SMD:SOT-23, F.Cu at (192.1, 27.2)
- added Q32: Q_NPN_BEC, Package_TO_SOT_SMD:SOT-23, F.Cu at (192.1, 31.7)
- added Q33: Q_NPN_BEC, Package_TO_SOT_SMD:SOT-23, F.Cu at (195.8, 27.1)
- added Q34: Q_NPN_BEC, Package_TO_SOT_SMD:SOT-23, F.Cu at (107.0, -158.8)
- added Q35: Q_NPN_BEC, Package_TO_SOT_SMD:SOT-23, F.Cu at (107.0, -154.3)
- added Q36: Q_NPN_BEC, Package_TO_SOT_SMD:SOT-23, F.Cu at (110.7, -159.0)
- added Q49: Q_NPN_BEC, Package_TO_SOT_SMD:SOT-23, F.Cu at (126.6, -158.8)
- added Q50: Q_NPN_BEC, Package_TO_SOT_SMD:SOT-23, F.Cu at (126.6, -154.3)
- added Q51: Q_NPN_BEC, Package_TO_SOT_SMD:SOT-23, F.Cu at (130.3, -159.0)
- added Q52: Q_NPN_BEC, Package_TO_SOT_SMD:SOT-23, F.Cu at (116.8, -143.4)
- added Q53: Q_NPN_BEC, Package_TO_SOT_SMD:SOT-23, F.Cu at (116.8, -139.0)
- added Q54: Q_NPN_BEC, Package_TO_SOT_SMD:SOT-23, F.Cu at (120.5, -143.6)
- added Q55: Q_NPN_BEC, Package_TO_SOT_SMD:SOT-23, F.Cu at (107.0, -143.4)
- added Q56: Q_NPN_BEC, Package_TO_SOT_SMD:SOT-23, F.Cu at (107.0, -139.0)
- added Q57: Q_NPN_BEC, Package_TO_SOT_SMD:SOT-23, F.Cu at (110.7, -143.6)
- added Q58: Q_NPN_BEC, Package_TO_SOT_SMD:SOT-23, F.Cu at (116.8, -158.8)
- added Q59: Q_NPN_BEC, Package_TO_SOT_SMD:SOT-23, F.Cu at (116.8, -154.3)
- added Q60: Q_NPN_BEC, Package_TO_SOT_SMD:SOT-23, F.Cu at (120.5, -159.0)
- added R16: 1k, Resistor_SMD:R_0402_1005Metric, F.Cu at (179.8, 33.7)
- added R20: 1k, Resistor_SMD:R_0402_1005Metric, F.Cu at (184.0, 33.7)
- added R24: 1k, Resistor_SMD:R_0402_1005Metric, F.Cu at (185.5, 27.4)
- added R28: 1k, Resistor_SMD:R_0402_1005Metric, F.Cu at (189.1, 26.2)
- added R32: 1k, Resistor_SMD:R_0402_1005Metric, F.Cu at (189.1, 30.5)
- added R36: 1k, Resistor_SMD:R_0402_1005Metric, F.Cu at (195.3, 32.0)
- added R40: 1k, Resistor_SMD:R_0402_1005Metric, F.Cu at (104.0, -159.8)
- added R44: 1k, Resistor_SMD:R_0402_1005Metric, F.Cu at (104.0, -155.5)
- added R48: 1k, Resistor_SMD:R_0402_1005Metric, F.Cu at (110.2, -154.0)
- added R49: 1k, Resistor_SMD:R_0402_1005Metric, F.Cu at (123.6, -159.8)
- added R50: 1k, Resistor_SMD:R_0402_1005Metric, F.Cu at (123.6, -155.5)
- added R51: 1k, Resistor_SMD:R_0402_1005Metric, F.Cu at (129.8, -154.0)
- added R52: 1k, Resistor_SMD:R_0402_1005Metric, F.Cu at (113.8, -144.4)
- added R53: 1k, Resistor_SMD:R_0402_1005Metric, F.Cu at (113.8, -140.2)
- added R54: 1k, Resistor_SMD:R_0402_1005Metric, F.Cu at (120.0, -138.7)
- added R55: 1k, Resistor_SMD:R_0402_1005Metric, F.Cu at (104.0, -144.4)
- added R56: 1k, Resistor_SMD:R_0402_1005Metric, F.Cu at (104.0, -140.2)
- added R57: 1k, Resistor_SMD:R_0402_1005Metric, F.Cu at (110.2, -138.7)
- added R58: 1k, Resistor_SMD:R_0402_1005Metric, F.Cu at (113.8, -159.8)
- added R59: 1k, Resistor_SMD:R_0402_1005Metric, F.Cu at (113.8, -155.5)
- added R60: 1k, Resistor_SMD:R_0402_1005Metric, F.Cu at (120.0, -154.0)
- moved Q25 180.3 mm to (137.8, -84.2)
- moved Q26 180.3 mm to (137.8, -79.8)
- moved Q27 180.3 mm to (141.5, -84.4)
- moved R12 180.3 mm to (141.1, -79.5)
- moved R4 180.3 mm to (134.8, -85.2)
- moved R8 180.3 mm to (134.8, -81.0)
- moved R2 62.4 mm to (159.9, 81.8)
- moved R6 62.4 mm to (159.9, 66.5)
- moved R1 62.2 mm to (159.9, 77.5)
- moved R5 62.2 mm to (159.9, 62.2)
- moved R3 56.2 mm to (166.2, 83.3)
- moved R7 56.2 mm to (166.2, 68.0)
- moved Q1 55.3 mm to (162.9, 63.2)
- moved Q13 55.3 mm to (162.9, 67.7)
- moved Q14 55.3 mm to (162.9, 83.0)
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Routing:
- net VCC: track 5.90 -> 129.2 mm, vias 0 -> 3
- net /SR-Latch1/!Q: track 0.00 -> 19.2 mm, vias 0 -> 2
- net GND: track 0.00 -> 8.22 mm, vias 0 -> 2
- net /SR-Latch1/Q: track 0.00 -> 7.90 mm, vias 0 -> 2
- net Net-(Q42-B): track 0.00 -> 6.13 mm
- net Net-(Q45-B): track 0.00 -> 6.13 mm
- net Net-(Q41-B): track 0.00 -> 6.13 mm
- net Net-(Q12-C): track 0.00 -> 6.13 mm
- net Net-(Q52-C): track 0.00 -> 6.13 mm
- net Net-(Q58-C): track 0.00 -> 6.13 mm
- net Net-(Q55-C): track 0.00 -> 6.13 mm
- net Net-(Q10-C): track 0.00 -> 6.13 mm
- net Net-(Q28-C): track 0.00 -> 6.13 mm
- net Net-(Q44-B): track 0.00 -> 6.13 mm
- net Net-(Q43-B): track 0.00 -> 6.13 mm
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